File: Board/csa_ultracpu.sch (EAGLE design)
At the start: 131 parts, among them IC1 RAMSOCK32TO512KSOP, IC10 RAMSOCK32TO512KSOP, IC11 74HCT574D, IC12 74HCT574D, IC13 74HCT244DW, IC14 74HCT14D, IC15 74HCT157D, IC18 74LS06D, IC19 74HCT244DW, IC2 74LS245DW, IC3 74LS245DW, IC4 74LS245DW, IC5 74LS245DW, IC6 74ACT138D, IC7 74LS245DW, IC8 MAX3421E, IC9 74LS166D, P1 CSABUS, Q2 32kHz, Q3 12MHz, X2 D-SUB15-HDR15RA

Commit message: update board to 1.3C
Parts:
- removed C28, C36, C37: 22u, rcl:CPOL-EUE2.5-6
- removed IC11, IC12: 74HCT574D, 74xx-eu:74HCT574D
- removed IC15: 74HCT157D, 74xx-eu:74HCT157D
- removed IC9: 74LS166D, 74xx-eu:74LS166D
- removed J1: (no value), con-amp:FLOPPY-4350211
- removed TO1: LM2937SOT-3.3V, csa:LM2937SOT
- added C100, C101, C102, C103, C104, C105, C109, C111, C112: 0.1u, rcl:C-EUC0603
- added C120, C121, C123: 1u, rcl:C-EUC0603
- added C63, C64, C65, C66, C67, C68, C69, C70, C71: 22u, rcl:C-EUC0805
- added D9: 1N4148, diode:DIODE-D-5
- added DS1818: DS1818, csa:DS1813
- added IC16: 74LVC8T245SO24, csa:74LVC8T245SO24
- added JP4, JP6: (no value), jumper:JP1E
- added JP5: (no value), jumper:JP2E
- added JS1: RENOSCXLH, csa:RENOSCXLH
- added R23, R24, R26: 10k, rcl:R-EU_0207/2V
- added R25: 4k7, rcl:R-EU_0207/2V
- added R27: 10k, rcl:R-EU_0204/5
- added R28, R31: 100, rcl:R-EU_0204/2V
- added R29: 330, rcl:R-EU_0207/2V
- added R30, R32: 680, rcl:R-EU_0204/2V
- added SJ1: (no value), jumper:SJ2W
- added SN1: MCP48X2, csa:MCP48X2
- added U$10, U$11, U$14, U$15, U$5, U$6, U$8: PESD5V0L1BA, csa:ESDBIDIR
- added U$16: AP2132B-1.2, csa:AP2132BB
- added U$17: AP2132B-2.5, csa:AP2132BB
- added U$18: SPIFLASH, csa:SPIFLASH
- added X1: SJ1-3513N, con-lumberg:1503_09
- C1, C14, C4: value 0.1u -> 1u
- C10: device rcl:C-EUC0603 -> rcl:C-EU050-025X075
- C106, C108, C11, C113: value 1u -> 0.1u
- C26: value 47u -> 0.1u; device rcl:CPOL-EUE2.5-6 -> rcl:C-EUC0603
- C3: value 0.1u -> 1u; device rcl:C-EUC0603 -> rcl:C-EU050-025X075
- C5: value 47u -> 22u; device rcl:CPOL-EUE5-6 -> rcl:C-EUC0805
- C57: value 22u -> 1u; device rcl:CPOL-EUE2.5-6 -> rcl:C-EUC0603
- IC14: value 74HCT14D -> 74LVC14
- IC18: value 74LS06D -> 74LVC06
- IC2, IC4, IC5: value 74LS245DW -> 74HCT245DW
- IC3: value 74LS245DW -> 74LS125D; device 74xx-eu:74LS245DW -> 74xx-eu:74LS125D
- IC6: value 74ACT138D -> 74HC138D
- IC7: value 74LS245DW -> 74S138D; device 74xx-eu:74LS245DW -> 74xx-eu:74S138D
- R12: value 1k -> 1k5
- U$2: value XC95288XLTQ144 -> XC3S250E; device csa:XC95288XLTQ144 -> csa:XC3S100E
- U$3: value DS1813 -> LDI1117; device csa:DS1813 -> csa:LDI1117
- renumbered C20 to C107, C50 to C106, C51 to C113, C52 to C110, C53 to C108
Connections:
- removed net /CHROMADDR: IC7A.G, U$2G$3.FB11MC12
- removed net /DENA: IC15A.G, U$2G$3.FB5MC14
- removed net /RAMCS: IC10G$1./CS, IC10G$1./OE, U$2G$3.FB10MC12
- removed net /SRLOAD: IC9A.SH/!LD, U$2G$3.FB7MC5
- removed net BG0: IC12A.5Q, IC15A.1A
- removed net BG1: IC12A.6Q, IC15A.2A
- removed net BG2: IC12A.7Q, IC15A.3A
- removed net BG3: IC12A.8Q, IC15A.4A
- removed net COLORLD: IC12A.CLK, U$2G$3.FB11MC5
- removed net COLORLD2: U$2G$3.FB2MC14
- removed net FA18: IC1G$1.A18, IC5A.B7, U$2G$3.FB14MC15
- removed net FG0: IC12A.1Q, IC15A.1B
- removed net FG1: IC12A.2Q, IC15A.2B
- removed net FG2: IC12A.3Q, IC15A.3B
- removed net FG3: IC12A.4Q, IC15A.4B
- removed net PHI2_IO: R5.1, U$2G$3.GCK2
- removed net PIXELS: IC15A.!A!/B, IC9A.QH
- removed net PXL0: IC11A.1Q, IC7A.B1, IC9A.A
- removed net PXL1: IC11A.2Q, IC7A.B2, IC9A.B
- removed net PXL2: IC11A.3Q, IC7A.B3, IC9A.C
- removed net PXL3: IC11A.4Q, IC7A.B4, IC9A.D
- removed net PXL4: IC11A.5Q, IC7A.B5, IC9A.E
- removed net PXL5: IC11A.6Q, IC7A.B6, IC9A.F
- removed net PXL6: IC11A.7Q, IC7A.B7, IC9A.G
- removed net PXL7: IC11A.8Q, IC7A.B8, IC9A.H
- removed net PXLLD: IC11A.CLK, U$2G$3.FB1MC15
- removed net RAMA11: IC10G$1.A11, IC7A.A8, U$2G$3.FB8MC3
- removed net RAMA3: IC10G$1.A3, U$2G$3.FB10MC11
- removed net RAMA5: IC10G$1.A5, IC7A.A2, U$2G$3.FB8MC5
- removed net RAMA9: IC10G$1.A9, IC7A.A6, U$2G$3.FB8MC8
- removed net SPI_IN1: IC8.MISO, U$13.SO, U$2G$3.FB10MC17, U$4.SO, U$9.MISO
- removed net SPI_OUT: IC8.MOSI, U$12.DI, U$13.SI, U$2G$3.FB9MC8, U$4.SI, U$9.MOSI
- removed net SRCLK: IC9A.CLK, U$2G$3.FB7MC3
- new net /FPGA_BOOT: IC7A.Y6, U$18./CS
- new net /LDAC: SN1./LDAC, U$2G$2.IO_L08N_0_VREF_0
- new net /RAMCS/M1: IC10G$1./CS, IC10G$1./OE, IC3B.O, U$2G$2.IO_60_M1
- new net 50MCAN: R12.2, R5.1, SJ1.3
- new net 50MSMD: JS1.OUT1, SJ1.1
- new net BV33: JP6.2, P1.VCC33
- new net DEBUG: U$2G$2.IO_L08P_0
- new net DONE: IC3A.OE, IC3B.OE, IC3C.OE, R29.1, U$1G$1.BE, U$2G$1.DONE
- new net FA18/HSWAP: IC1G$1.A18, IC3A.O, IC5A.B7, U$2G$2.IO_L10N_0_HSWAP
- new net GRAPHIC5V: IC18F.I, JP1.1
- new net INIT_B: U$2G$2.IO_L01N_2_INIT_B
- new net M2: IC3C.O, U$2G$2.IP_L06N_2_M2_GCLK1
- new net N$12: R24.1, U$16.PG
- new net N$21: D9.C, JP1.2, R26.2
- new net N$22: R28.1, SN1.VOUTB
- new net N$23: C3.2, R30.2, X1.2
- new net N$26: R31.1, SN1.VOUTA
- new net N$27: C10.1, JP5.1, R31.2
- new net N$28: C10.2, R32.2, X1.3
- new net N$42: C3.1, JP5.3, R28.2
- new net N$6: R23.1, U$17.PG
- new net N$7: QG1.OUT, R5.2
- new net PROG_B: JP4.2, R25.1, U$2G$1.PROG_B
- new net RAMA11/VS2: IC10G$1.A11, U$2G$2.IO_L09P_2_VS2_A19
- new net RAMA3/M0: IC10G$1.A3, U$2G$2.IO_L08P_2_M0
- new net RAMA5/VS1: IC10G$1.A5, U$2G$2.IO_L09N_2_VS1_A18
- new net RAMA9/VS0: IC10G$1.A9, U$2G$2.IO_L10P_2_VS0_A17
- new net SPISELA/CSO_B: IC7A.A, U$2G$2.IO_L01P_2_CSO_B
- new net SPISELB: IC7A.B, U$2G$2.IO_L08N_3
- new net SPISELC: IC7A.C, U$2G$2.IO_L08P_3
- new net SPI_ACLK: SN1.SCK, U$2G$2.IO_L05N_3_LHCLK3
- new net SPI_AMOSI: SN1.SDI, U$2G$2.IO_L05P_3_LHCLK2
- new net SPI_CLK/CCLK: U$18.SCK, U$2G$2.IO_L10N_2_CCLK
- new net SPI_MISO/DIN: IC8.MISO, U$13.SO, U$18.SO, U$2G$2.IO_L08N_2_DIN_D0, U$4.SO, U$9.MISO
- new net SPI_MOSI: IC8.MOSI, U$12.DI, U$13.SI, U$18.SI, U$2G$2.IO_L02N_2_MOSI_CSI_B, U$4.SI, U$9.MOSI
- new net SPI_NAUDIO: SN1./CS, U$2G$2.IO_L02P_0
- new net V12: C102.2, C105.2, C108.2, C111.2, C57.2, C66.1, U$16.VOUT, U$2G$1.VCCINT@0, U$2G$1.VCCINT@1, U$2G$1.VCCINT@2, U$2G$1.VCCINT@3
- new net V25: C101.1, C104.1, C109.1, C112.1, C121.1, C123.1, C64.1, R25.2, U$16.EN, U$17.VOUT, U$2G$1.VCCAUX@0, U$2G$1.VCCAUX@1, U$2G$1.VCCAUX@2, U$2G$1.VCCAUX@3, U$7G$2.VCC
- net /BE_DOUT: now also IC16./OE, U$2G$2.IO_L07N_0_GCLK11; no longer IC3A.G, U$2G$3.FB1MC6
- net /BE_OUT: now also U$2G$2.IO_L07P_0_GCLK10; no longer U$2G$3.FB11MC10
- net /FRAMSEL: now also U$2G$2.IO_124_VREF_0; no longer U$2G$3.GTS2
- net /IOSEL: now also U$2G$2.IO_132; no longer U$2G$3.FB11MC14
- net /IRQ: now also U$2G$2.IO_L07P_3_LHCLK6
- net /MEMSEL: now also U$2G$2.IO_L01P_0; no longer U$2G$3.FB1MC14
- net /RAMWE: now also U$2G$2.IO_L03N_1_A11; no longer U$2G$3.FB5MC17
- net /RES: now also DS1818./RESET, U$2G$2.IO_L02N_0; no longer U$2G$3.GSR, U$3./RESET
- net 50M: now also SJ1.2, U$2G$2.IO_L04P_0_GCLK4; no longer QG1.OUT, U$2G$3.GCK0
- net A0: now also U$2G$2.IP_18; no longer U$2G$3.FB14MC10
- net A1: now also U$2G$2.IP_L06P_2_RDWR_B_GCLK0; no longer U$2G$3.FB14MC8
- net A10: now also U$2G$2.IP_12_VREF_3; no longer U$2G$3.FB16MC5
- net A11: now also U$2G$2.IP_141; no longer U$2G$3.FB16MC3
- net A12: now also U$2G$2.IP_L06P_0_GCLK8; no longer U$2G$3.FB16MC2
- net A13: now also U$2G$2.IP_136; no longer U$2G$3.FB15MC15
- net A14: now also U$2G$2.IP_L03N_0; no longer U$2G$3.FB15MC17
- net A15: now also U$2G$2.IP_L06N_0_GCLK9; no longer U$2G$3.FB15MC12
- net A2: now also U$2G$2.IP_L03N_2_VREF_2; no longer U$2G$3.FB14MC6
- net A3: now also U$2G$2.IP_41; no longer U$2G$3.FB14MC5
- net A4: now also U$2G$2.IP_L03P_2; no longer U$2G$3.FB14MC3
- net A5: now also U$2G$2.IP_36; no longer U$2G$3.FB16MC12
- net A6: now also U$2G$2.IP_38; no longer U$2G$3.FB16MC11
- net A7: now also U$2G$2.IP_24; no longer U$2G$3.FB16MC10
- net A8: now also U$2G$2.IP_29; no longer U$2G$3.FB16MC8
- net A9: now also U$2G$2.IP_10; no longer U$2G$3.FB16MC6
- net BD0: now also IC16.A1; no longer IC3A.A1
- net BD1: now also IC16.A2; no longer IC3A.A2
- net BD2: now also IC16.A3; no longer IC3A.A3
- net BD3: now also IC16.A4; no longer IC3A.A4
- net BD4: now also IC16.A5; no longer IC3A.A5
- net BD5: now also IC16.A6; no longer IC3A.A6
- net BD6: now also IC16.A7; no longer IC3A.A7
- net BD7: now also IC16.A8; no longer IC3A.A8
- net BE_IN: now also U$2G$2.IP_L03P_0; no longer U$2G$3.FB6MC10
- net BOUT: now also U$2G$2.IO_L07P_1_A4_RHCLK6; no longer IC15A.2Y
- net C2PHI2: now also U$2G$2.IO_L10N_1_LDC2; no longer U$2G$3.FB1MC8
- net C8PHI2: now also U$2G$2.IO_L10P_1_LDC1; no longer U$2G$3.FB1MC10
- net CPHI2: now also U$2G$2.IO_L01N_0; no longer U$2G$3.FB1MC12
- net D0: now also IC16.B1, U$2G$2.IO_L01N_3; no longer IC3A.B1, U$2G$3.FB15MC14
- net D1: now also IC16.B2, U$2G$2.IO_L01P_3; no longer IC3A.B2, U$2G$3.FB15MC11
- net D2: now also IC16.B3, U$2G$2.IO_L04N_3_LHCLK1; no longer IC3A.B3, U$2G$3.FB15MC10
- net D3: now also IC16.B4, U$2G$2.IO_L02P_3; no longer IC3A.B4, U$2G$3.FB15MC8
- net D4: now also IC16.B5, U$2G$2.IO_L04P_3_LHCLK0; no longer IC3A.B5, U$2G$3.FB15MC3
- net D5: now also IC16.B6, U$2G$2.IO_L03P_3; no longer IC3A.B6, U$2G$3.FB15MC2
- net D6: now also IC16.B7, U$2G$2.IO_L03N_3; no longer IC3A.B7, U$2G$3.FB13MC17
- net D7: now also IC16.B8, U$2G$2.IO_L02N_3_VREF_3; no longer IC3A.B8, U$2G$3.FB13MC15
- net E: now also U$2G$2.IO_L06P_3_LHCLK4; no longer U$2G$3.FB6MC14
- net EXTIO: now also U$2G$2.IP_114; no longer U$2G$3.FB10MC14
- net FA15: now also U$2G$2.IO_L09P_0; no longer U$2G$3.FB13MC2
- net FA16: now also U$2G$2.IO_L09N_0; no longer U$2G$3.FB14MC11
- net FA17: now also U$2G$2.IO_L10P_0; no longer U$2G$3.FB14MC14
- net FA19: now also U$2G$2.IO_L09N_1_LDC0; no longer U$2G$3.GTS3
- net GND: now also C100.1, C101.2, C102.1, C103.2, C104.2, C105.1, C109.2, C111.1, C112.2, C120.2, C121.2, C123.2, C26.1, C5.2, C57.1, C63.2, C64.2, C65.2, C66.2, C67.2, C68.2, C69.2, C70.2, C71.2, DS1818.GND, IC14P.GND, IC16.GND@1, IC16.GND@2, IC16.GND@3, IC18P.GND, IC1G$2.GND, IC3A.I, IC3B.I, IC3C.I, IC3P.GND, IC6P.GND, IC7A.G2A, IC7A.G2B, IC7P.GND, JP4.1, JP5.2, JS1.VSS, R12.1, R26.1, R30.1, R32.1, SN1.GND, U$10.2, U$11.2, U$14.2, U$15.2, U$16.ADJ, U$16.GND, U$17.ADJ, U$17.GND, U$18.GND, U$2G$1.GND@0, U$2G$1.GND@1, U$2G$1.GND@10, U$2G$1.GND@11, U$2G$1.GND@12, U$2G$1.GND@2, U$2G$1.GND@3, U$2G$1.GND@4, U$2G$1.GND@5, U$2G$1.GND@6, U$2G$1.GND@7, U$2G$1.GND@8, U$2G$1.GND@9, U$5.2, U$6.2, U$8.2, X1.1; no longer C10.1, C26.-, C28.-, C3.2, C36.-, C37.-, C5.-, C57.-, IC11A.OC, IC12A.OC, IC7A.DIR, IC9A.INH, J1.2, J1.3, TO1.GND, U$2G$2.GND@0, U$2G$2.GND@1, U$2G$2.GND@10, U$2G$2.GND@11, U$2G$2.GND@12, U$2G$2.GND@2, U$2G$2.GND@3, U$2G$2.GND@4, U$2G$2.GND@5, U$2G$2.GND@6, U$2G$2.GND@7, U$2G$2.GND@8, U$2G$2.GND@9
- net GOUT: now also U$2G$2.IO_L07N_1_A3_RHCLK7; no longer IC15A.3Y
- net GRAPHIC: now also IC18F.O, R27.1, U$2G$2.IP_107; no longer JP1.1, U$2G$3.FB11MC17
- net HSYNC: now also U$2G$2.IO_98_A0; no longer U$2G$3.FB7MC12
- net IOINH: now also U$2G$2.IP_111; no longer U$2G$3.FB10MC2
- net IOUT: now also U$2G$2.IO_L06N_1_A5_RHCLK5; no longer IC15A.1Y
- net N$17: now also U$8.1
- net N$18: now also U$10.1
- net N$19: now also U$11.1
- net N$24: now also U$6.1
- net N$25: now also U$5.1
- net N$35: now also U$14.1
- net N$36: now also U$15.1
- net PET_VSYNC: now also D9.A, U$2G$2.IO_L06P_1_A6_RHCLK4; no longer JP1.2, U$2G$3.FB5MC15
- net PHI2: now also U$2G$2.IO_L05N_0_GCLK7; no longer R12.2, U$2G$3.FB9MC12
- net R/-W: now also IC16.DIR, U$2G$2.IO_L05P_0_GCLK6; no longer IC3A.DIR, U$2G$3.FB1MC5
- net RAMA0: now also U$2G$2.IO_52_D5; no longer U$2G$3.FB10MC5
- net RAMA1: now also U$2G$2.IO_L05N_2_D3_GCLK15; no longer U$2G$3.FB10MC6
- net RAMA10: now also U$2G$2.IO_L07P_2_D2_GCLK2; no longer IC7A.A7, U$2G$3.FB10MC10
- net RAMA12: now also U$2G$2.IO_L03P_1_A12; no longer U$2G$3.FB6MC6
- net RAMA13: now also U$2G$2.IO_L02N_1_A13; no longer U$2G$3.FB6MC5
- net RAMA14: now also U$2G$2.IO_83_VREF_1; no longer U$2G$3.FB4MC14
- net RAMA15: now also U$2G$2.IO_L05P_1_A8_RHCLK2; no longer U$2G$3.FB2MC3
- net RAMA16: now also U$2G$2.IO_L04N_1_A9_RHCLK1; no longer U$2G$3.FB2MC2
- net RAMA17: now also U$2G$2.IO_L04P_1_A10_RHCLK0; no longer U$2G$3.FB4MC6
- net RAMA18: now also U$2G$2.IO_L05N_1_A7_RHCLK3; no longer U$2G$3.FB2MC5
- net RAMA2: now also U$2G$2.IO_L07N_2_D1_GCLK3; no longer U$2G$3.FB10MC8
- net RAMA4: now also U$2G$2.IO_66_VREF_2; no longer IC7A.A1, U$2G$3.FB8MC2
- net RAMA6: now also U$2G$2.IO_L01P_1_A16; no longer IC7A.A3, U$2G$3.FB8MC10
- net RAMA7: now also U$2G$2.IO_L02P_1_A14; no longer IC7A.A4, U$2G$3.FB6MC3
- net RAMA8: now also U$2G$2.IO_L01N_1_A15; no longer IC7A.A5, U$2G$3.FB6MC2
- net RAMD0: now also U$2G$2.IO_L04P_2_D7_GCLK12; no longer IC11A.1D, IC12A.1D, U$2G$3.FB12MC12
- net RAMD1: now also U$2G$2.IO_L02P_2_DOUT_BUSY; no longer IC11A.2D, IC12A.2D, U$2G$3.FB12MC8
- net RAMD2: now also U$2G$2.IO_L10N_3; no longer IC11A.3D, IC12A.3D, U$2G$3.FB12MC3
- net RAMD3: now also U$2G$2.IO_L09P_3; no longer IC11A.4D, IC12A.4D, U$2G$3.FB12MC2
- net RAMD4: now also U$2G$2.IO_L09N_3; no longer IC11A.5D, IC12A.5D, U$2G$3.FB12MC5
- net RAMD5: now also U$2G$2.IO_L10P_3; no longer IC11A.6D, IC12A.6D, U$2G$3.FB12MC10
- net RAMD6: now also U$2G$2.IO_L04N_2_D6_GCLK13; no longer IC11A.7D, IC12A.7D, U$2G$3.FB9MC14
- net RAMD7: now also U$2G$2.IO_L05P_2_D4_GCLK14; no longer IC11A.8D, IC12A.8D, U$2G$3.FB9MC17
- net RDY: now also U$2G$2.IO_31_VREF_3
- net ROUT: now also U$2G$2.IO_L08P_1_A2; no longer IC15A.4Y
- net SPI_CLK: now also U$2G$2.IO_L09P_1_HDC; no longer U$2G$3.FB9MC2
- net SPI_IN3: now also U$2G$2.IP_69; no longer U$2G$3.FB10MC3
- net SPI_NFLASH: now also IC7A.Y1; no longer U$2G$3.FB9MC5
- net SPI_NSEL2: now also IC7A.Y2; no longer U$2G$3.FB5MC2
- net SPI_NSEL3: now also IC7A.Y3; no longer U$2G$3.FB5MC10
- net SPI_NSEL4: now also IC7A.Y4; no longer U$2G$3.FB5MC12
- net SPI_NSEL5: now also IC7A.Y5; no longer U$2G$3.FB11MC3
- net SYNC: now also U$2G$2.IO_L04N_0_GCLK5; no longer U$2G$3.FB1MC17
- net TCK: now also U$2G$3.TCK; no longer U$2G$1.TCK
- net TDI: now also U$2G$3.TDI; no longer U$2G$1.TDI
- net TDO: now also U$2G$3.TDO; no longer U$2G$1.TDO
- net TMS: now also U$2G$3.TMS; no longer U$2G$1.TMS
- net V33: now also C100.2, C103.1, C107.2, C120.1, C14.1, C17.1, C18.1, C22.2, C24.2, C25.2, C26.2, C31.2, C32.2, C35.2, C48.2, C5.1, C54.2, C55.2, C56.2, DS1818.VCC, IC10G$2.VCC, IC14P.VCC, IC16.VCCB@1, IC16.VCCB@2, IC18P.VCC, IC1G$2.VCC, IC3P.VCC, IC7A.G1, IC7P.VCC, JP6.1, JS1.VDD, R10.1, R11.1, R27.2, R29.2, SN1.VCC, U$18./HOLD, U$18.VCC, U$1G$1.VDD, U$1G$2.VCC, U$2G$1.VCCO_0@0, U$2G$1.VCCO_0@1, U$2G$1.VCCO_1@0, U$2G$1.VCCO_1@1, U$2G$1.VCCO_2@0, U$2G$1.VCCO_2@1, U$2G$1.VCCO_2@2, U$2G$1.VCCO_3@0, U$2G$1.VCCO_3@1, U$3.VO; no longer C10.2, C108.2, C3.1, C5.+, TO1.VO, U$2G$2.VCC@0, U$2G$2.VCC@1, U$2G$2.VCC@2, U$2G$2.VCC@3, U$2G$2.VIO@0, U$2G$2.VIO@1, U$2G$2.VIO@2, U$2G$2.VIO@3, U$2G$2.VIO@4, U$2G$2.VIO@5, U$7G$2.VCC
- net VCC: now also C63.1, C65.1, C67.1, C68.1, C69.1, C70.1, C71.1, IC16.VCCA, IC6P.VCC, R23.2, R24.2, U$16.VCTRL, U$16.VIN, U$17.EN, U$17.VCTRL, U$17.VIN, U$3.VI; no longer C107.2, C14.1, C17.1, C18.1, C22.2, C24.2, C25.2, C26.+, C28.+, C31.2, C32.2, C35.2, C36.+, C37.+, C48.2, C54.2, C55.2, C56.2, C57.+, IC10G$2.VCC, IC9A.CLR, IC9A.SER, J1.4, R10.1, R11.1, R12.1, R5.2, TO1.VI, U$1G$1.BE, U$1G$1.VDD, U$1G$2.VCC, U$3.VCC
- net VDA: now also U$2G$2.IO_L06N_3_LHCLK5; no longer U$2G$3.FB13MC11
- net VPA: now also U$2G$2.IO_L07N_3_LHCLK7; no longer U$2G$3.FB13MC8
- net VPB: now also U$2G$2.IP_6
- net VSYNC: now also U$2G$2.IO_L08N_1_A1; no longer U$2G$3.FB7MC15
Other:
- note added: "1000mA, according to LDI1117 datasheet (linear regulator though)"
- note added: "3.3V side"
- note added: "5V side"
- note added: "CSA-ULTRACPU-V1.1A-20220820"
- note added: "CSA-ULTRACPU-V1.3B-20230811"
- note added: "CSA-ULTRACPU-V1.3C"
- note added: "CSA-ULTRACPU-V1.3C-20231105"
- note added: "CSA-ULTRACPU-V1.3C-20231117"
- note added: "CSA-UTRACPU-V1.3C"
- note added: "DS1818"
- note added: "For Master SPI config, M[0..2] need to be 001 (M0=1, M1=0, M2=0) - doing this with '125 when DONE is low VS[0..2] select Flash variant M[] and VS[] are sampled when INIT_B goes high, std I/O after config DONE goes high after initialization is finished. Boot PROM connections: MOSI is SPI MOSI DIN is SPI MISO CSO_B is Boot flash /select CCLK is SPI clock (CCLK is 50 Ohm transmission line - no branc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"
- note added: "HSWAP pulldown during configuration to enable pullups on config+I/O pins"
- note added: "Protection against accidently connecting the wrong way around"
- note added: "V1.0B: - Added "Brown Fix" V1.1A: - 3.3/5V level converter - VGA ESD protection diodes"
- note added: "V1.1A: - 3.3V IC families V1.3A: - pull color logic into FPGA V1.3B: - add audio output via MCP4802 V1.3C - stereo jack to get out both channels"
- note added: "V1.1A: - 3.3V/5V level converter V1.2A: - use 74LVC06 instead of HCT - voltage conversion for GRAPHIC V1.2B: - pullup for GRAPHIC V1.3C: - jumper for 3.3V on Bus"
- note added: "V1.1A: - added USB ESD protection diodes"
- note added: "V1.2A: - Spartan 3E instead of XC95288 V1.2B: - add missing VCCO supply - Pulldown for VSYNC V1.3B: - pull colur handling into FPGA - re-layout - add 70MHz SMD oscillator option - fix FPGA boot, add FPGA boot prom - add /IRQ to FPGA output V1.3C: - move R/-W around to document patch in 1.3B"
- note added: "V1.2B: - fix pinout of LDI1117 V1.3B: - adapt C values"
- note added: "Voltage divider 5V to 3.3V"
- note removed: "400/500mA, according to LM2937 datasheet"
- note removed: "CSA-ULTRACPU-V1.0A"
- note removed: "CSA-ULTRACPU-V1.0A-20210927"
- note removed: "CSA-ULTRACPU-V1.0B"
- note removed: "CSA-ULTRACPU-V1.0B-20220409"
- note removed: "CSA-ULTRACPU-V1.0B-20220418"
- note removed: "CSA-UTRACPU-V1.0B"
- note removed: "Char & Pixel"
- note removed: "Color"
- note removed: "Read Charrom"
- note removed: "V1.0B: - Added "Brown Fix""
- note removed: "V1.0B: - Remove second color buffer - re-order color outputs to as in C128 VDC - fixed swapped A/B and G inputs to IC15 - swapped FG and BG colors ... SR output =1 for FG(!)"
- note removed: "V1.0B: - turn JP1 180 degrees so it confirms with CSA CPU and PETIO"

Commit message: update board to 2.0b from internal repo
Parts:
- removed C23: 0.1u, rcl:C-EUC0603
- removed C63: 22u, rcl:C-EUC0805
- removed QG2: 16MHz, crystal:CRYSTAL_RES-SG51
- removed R21: 2k, rcl:R-EU_0204/2V
- removed R23: 10k, rcl:R-EU_0207/2V
- removed R3: 10k, rcl:R-EU_0204/2V
- removed U$17: AP2132B-2.5, csa:AP2132BB
- added C20, C28, C36, C37: 0.1u, rcl:C-EUC0603
- added D10: 1N4148DO35-7, diode:1N4148DO35-7
- added JP10, JP11, JP8, JP9: PIN, csa:PIN
- IC3: value 74LS125D -> 74LVC125
- IC6: value 74HC138D -> 74LVC1G04DBV; device 74xx-eu:74ACT138D -> 74xx-little-us:74LVC1G04DBV
- IC7: value 74S138D -> 74LVC138
- U$2: value XC3S250E -> XC6SLX9-TQG144; device csa:XC3S100E -> csa:XC9SLX9-TQG144
Connections:
- removed net /RAMCS/M1: IC10G$1./CS, IC10G$1./OE, IC3B.O, U$2G$2.IO_60_M1
- removed net C16M: IC19A.A2, QG2.OUT
- removed net DEBUG: U$2G$2.IO_L08P_0
- removed net INIT_B: U$2G$2.IO_L01N_2_INIT_B
- removed net INTENSITY: D7.A, IC2A.B4, IC6A.G2B
- removed net IOUT: IC2A.A4, U$2G$2.IO_L06N_1_A5_RHCLK5
- removed net M2: IC3C.O, U$2G$2.IP_L06N_2_M2_GCLK1
- removed net N$1: IC2A.A7, IC2A.A8, R3.2
- removed net N$6: R23.1, U$17.PG
- removed net RAMA11/VS2: IC10G$1.A11, U$2G$2.IO_L09P_2_VS2_A19
- removed net RAMA3/M0: IC10G$1.A3, U$2G$2.IO_L08P_2_M0
- removed net RAMA5/VS1: IC10G$1.A5, U$2G$2.IO_L09N_2_VS1_A18
- removed net RAMA9/VS0: IC10G$1.A9, U$2G$2.IO_L10P_2_VS0_A17
- removed net SPI_CLK: IC8.SCLK, U$12.SCK, U$13.SCK, U$2G$2.IO_L09P_1_HDC, U$4.SCK, U$9.SCK
- removed net V25: C101.1, C104.1, C109.1, C112.1, C121.1, C123.1, C64.1, R25.2, U$16.EN, U$17.VOUT, U$2G$1.VCCAUX@0, U$2G$1.VCCAUX@1, U$2G$1.VCCAUX@2, U$2G$1.VCCAUX@3, U$7G$2.VCC
- new net /BE: IC6A.I, U$2G$1.IO_L33P_1
- new net /RAMCS: IC10G$1./CS, IC10G$1./OE, U$2G$1.IO_L13N_D10_2
- new net BE: IC6A.O, U$1G$1.BE
- new net IBLUE: D7.A, IC2A.B4
- new net IBOUT: IC2A.A4, U$2G$1.IO_L41P_GCLK9_IRDY1_1
- new net IGOUT: IC2A.A7, U$2G$1.IO_L74N_DOUT_BUSY_1
- new net IGREEN: D1.A, IC2A.B7
- new net IRED: D10.A, IC2A.B8
- new net IROUT: IC2A.A8, U$2G$1.IO_L1P_1
- new net RAMA11: IC10G$1.A11, U$2G$1.IO_L12P_D1_MISO2_2
- new net RAMA3: IC10G$1.A3, IC3B.O, U$2G$1.IO_L13P_M1_2
- new net RAMA5: IC10G$1.A5, U$2G$1.IO_L2N_CMPMOSI_2
- new net RAMA9: IC10G$1.A9, U$2G$1.IO_L1N_M0_CMPMISO_2
- net /BE_DOUT: now also U$2G$1.IO_L34N_GCLK18_0; no longer U$2G$2.IO_L07N_0_GCLK11
- net /BE_OUT: now also U$2G$1.IO_L35P_GCLK17_0; no longer U$2G$2.IO_L07P_0_GCLK10
- net /FRAMSEL: now also U$2G$1.IO_L62N_VREF_0; no longer U$2G$2.IO_124_VREF_0
- net /IOSEL: now also U$2G$1.IO_L34P_GCLK19_0; no longer U$2G$2.IO_132
- net /IRQ: now also JP11.1, U$2G$1.IO_L41N_GCLK26_3; no longer U$2G$2.IO_L07P_3_LHCLK6
- net /LDAC: now also U$2G$1.IO_L4P_0; no longer U$2G$2.IO_L08N_0_VREF_0
- net /MEMSEL: now also U$2G$1.IO_L66P_SCP1_0; no longer U$2G$2.IO_L01P_0
- net /RAMWE: now also U$2G$1.IO_L45N_1; no longer U$2G$2.IO_L03N_1_A11
- net /RES: now also IC3C.O, U$2G$1.IO_L64P_SCP5_0; no longer U$2G$2.IO_L02N_0
- net 50M: now also U$2G$1.IO_L37N_GCLK12_0; no longer U$2G$2.IO_L04P_0_GCLK4
- net A0: now also U$2G$1.IO_L43P_GCLK23_3; no longer U$2G$2.IP_18
- net A1: now also U$2G$1.IO_L30P_GCLK1_D13_2; no longer U$2G$2.IP_L06P_2_RDWR_B_GCLK0
- net A10: now also U$2G$1.IO_L49N_3; no longer U$2G$2.IP_12_VREF_3
- net A11: now also U$2G$1.IO_L2P_0; no longer U$2G$2.IP_141
- net A12: now also U$2G$1.IO_L36P_GCLK15_0; no longer U$2G$2.IP_L06P_0_GCLK8
- net A13: now also U$2G$1.IO_L3N_0; no longer U$2G$2.IP_136
- net A14: now also U$2G$1.IO_L63P_SCP7_0; no longer U$2G$2.IP_L03N_0
- net A15: now also U$2G$1.IO_L35N_GCLK16_0; no longer U$2G$2.IP_L06N_0_GCLK9
- net A2: now also U$2G$1.IO_L49N_D4_2; no longer U$2G$2.IP_L03N_2_VREF_2
- net A3: now also U$2G$1.IO_L62N_D6_2; no longer U$2G$2.IP_41
- net A4: now also U$2G$1.IO_L62P_D5_2; no longer U$2G$2.IP_L03P_2
- net A5: now also U$2G$1.IO_L64N_D9_2; no longer U$2G$2.IP_36
- net A6: now also U$2G$1.IO_L64P_D8_2; no longer U$2G$2.IP_38
- net A7: now also U$2G$1.IO_L37N_3; no longer U$2G$2.IP_24
- net A8: now also U$2G$1.IO_L36P_3; no longer U$2G$2.IP_29
- net A9: now also U$2G$1.IO_L50P_3; no longer U$2G$2.IP_10
- net BE_IN: now also U$2G$1.IO_L63N_SCP6_0; no longer U$2G$2.IP_L03P_0
- net BLUE: no longer IC6A.G2A
- net BOUT: now also U$2G$1.IO_L40N_GCLK10_1; no longer U$2G$2.IO_L07P_1_A4_RHCLK6
- net C2PHI2: now also U$2G$1.IO_L1N_VREF_1; no longer U$2G$2.IO_L10N_1_LDC2
- net C8PHI2: now also U$2G$1.IO_L32P_1; no longer U$2G$2.IO_L10P_1_LDC1
- net CPHI2: now also U$2G$1.IO_L65N_SCP2_0; no longer U$2G$2.IO_L01N_0
- net D0: now also U$2G$1.IO_L83P_3; no longer U$2G$2.IO_L01N_3
- net D1: now also U$2G$1.IO_L83N_VREF_3; no longer U$2G$2.IO_L01P_3
- net D2: now also U$2G$1.IO_L44N_GCLK20_3; no longer U$2G$2.IO_L04N_3_LHCLK1
- net D3: now also U$2G$1.IO_L52N_3; no longer U$2G$2.IO_L02P_3
- net D4: now also U$2G$1.IO_L49P_3; no longer U$2G$2.IO_L04P_3_LHCLK0
- net D5: now also U$2G$1.IO_L51P_3; no longer U$2G$2.IO_L03P_3
- net D6: now also U$2G$1.IO_L50N_3; no longer U$2G$2.IO_L03N_3
- net D7: now also U$2G$1.IO_L52P_3; no longer U$2G$2.IO_L02N_3_VREF_3
- net DONE: now also U$2G$2.DONE_2; no longer U$1G$1.BE, U$2G$1.DONE
- net E: now also U$2G$1.IO_L42N_GCLK24_3; no longer U$2G$2.IO_L06P_3_LHCLK4
- net EXTIO: now also U$2G$1.IO_L65P_SCP3_0; no longer U$2G$2.IP_114
- net FA15: now also U$2G$1.IO_L3P_0; no longer U$2G$2.IO_L09P_0
- net FA16: now also U$2G$1.IO_L2N_0; no longer U$2G$2.IO_L09N_0
- net FA17: now also U$2G$1.IO_L1N_VREF_0; no longer U$2G$2.IO_L10P_0
- net FA18/HSWAP: now also U$2G$1.IO_L1P_HSWAPEN_0; no longer U$2G$2.IO_L10N_0_HSWAP
- net FA19: now also U$2G$1.IO_L32N_1; no longer U$2G$2.IO_L09N_1_LDC0
- net GND: now also C20.2, C28.2, C36.2, C37.2, U$2G$2.GND, U$2G$2.GND@1, U$2G$2.GND@10, U$2G$2.GND@11, U$2G$2.GND@12, U$2G$2.GND@2, U$2G$2.GND@3, U$2G$2.GND@4, U$2G$2.GND@5, U$2G$2.GND@6, U$2G$2.GND@7, U$2G$2.GND@8, U$2G$2.GND@9; no longer C23.1, C63.2, QG2.VSS, R3.1, U$17.ADJ, U$17.GND, U$2G$1.GND@0, U$2G$1.GND@1, U$2G$1.GND@10, U$2G$1.GND@11, U$2G$1.GND@12, U$2G$1.GND@2, U$2G$1.GND@3, U$2G$1.GND@4, U$2G$1.GND@5, U$2G$1.GND@6, U$2G$1.GND@7, U$2G$1.GND@8, U$2G$1.GND@9
- net GOUT: now also U$2G$1.IO_L40P_GCLK11_1; no longer U$2G$2.IO_L07N_1_A3_RHCLK7
- net GRAPHIC: now also U$2G$1.IO_L4N_0; no longer U$2G$2.IP_107
- net GREEN: no longer IC6A.C
- net HSYNC: now also U$2G$1.IO_L33N_1; no longer U$2G$2.IO_98_A0
- net IOINH: now also U$2G$1.IO_L66N_SCP0_0; no longer U$2G$2.IP_111
- net N$11: now also IC19A.A2
- net N$14: now also D1.C; no longer D7.C, R18.1, R20.1
- net N$16: now also D7.C, R18.1; no longer IC6A.Y7, R21.1
- net N$18: no longer D1.A
- net N$20: now also D10.C, R20.1; no longer D1.C, R21.2
- net PET_VSYNC: now also U$2G$1.IO_L41N_GCLK8_1; no longer U$2G$2.IO_L06P_1_A6_RHCLK4
- net PHI2: now also JP9.1, U$2G$1.IO_L36N_GCLK14_0; no longer U$2G$2.IO_L05N_0_GCLK7
- net PROG_B: now also U$2G$2.PROGRAM_B_2; no longer U$2G$1.PROG_B
- net R/-W: now also U$2G$1.IO_L37P_GCLK13_0; no longer U$2G$2.IO_L05P_0_GCLK6
- net RAMA0: now also U$2G$1.IO_L31N_GCLK30_D15_2; no longer U$2G$2.IO_52_D5
- net RAMA1: now also U$2G$1.IO_L30N_GCLK0_USERCCLK_2; no longer U$2G$2.IO_L05N_2_D3_GCLK15
- net RAMA10: now also U$2G$1.IO_L14N_D12_2; no longer U$2G$2.IO_L07P_2_D2_GCLK2
- net RAMA12: now also U$2G$1.IO_L46P_1; no longer U$2G$2.IO_L03P_1_A12
- net RAMA13: now also U$2G$1.IO_L46N_1; no longer U$2G$2.IO_L02N_1_A13
- net RAMA14: now also U$2G$1.IO_L45P_1; no longer U$2G$2.IO_83_VREF_1
- net RAMA15: now also U$2G$1.IO_L42N_GCLK6_TRDY1_1; no longer U$2G$2.IO_L05P_1_A8_RHCLK2
- net RAMA16: now also U$2G$1.IO_L43P_GCLK5_1; no longer U$2G$2.IO_L04N_1_A9_RHCLK1
- net RAMA17: now also U$2G$1.IO_L43N_GCLK4_1; no longer U$2G$2.IO_L04P_1_A10_RHCLK0
- net RAMA18: now also U$2G$1.IO_L42P_GCLK7_1; no longer U$2G$2.IO_L05N_1_A7_RHCLK3
- net RAMA2: now also U$2G$1.IO_L14P_D11_2; no longer U$2G$2.IO_L07N_2_D1_GCLK3
- net RAMA4: now also U$2G$1.IO_L12N_D2_MISO3_2; no longer U$2G$2.IO_66_VREF_2
- net RAMA6: now also U$2G$1.IO_L74P_AWAKE_1; no longer U$2G$2.IO_L01P_1_A16
- net RAMA7: now also U$2G$1.IO_L47P_1; no longer U$2G$2.IO_L02P_1_A14
- net RAMA8: now also U$2G$1.IO_L47N_1; no longer U$2G$2.IO_L01N_1_A15
- net RAMD0: now also U$2G$1.IO_L48N_RDRW_B_VREF_2; no longer U$2G$2.IO_L04P_2_D7_GCLK12
- net RAMD1: now also U$2G$1.IO_L49P_D3_2; no longer U$2G$2.IO_L02P_2_DOUT_BUSY
- net RAMD2: now also U$2G$1.IO_L65P_INIT_B_2; no longer U$2G$2.IO_L10N_3
- net RAMD3: now also U$2G$1.IO_L2P_3; no longer U$2G$2.IO_L09P_3
- net RAMD4: now also U$2G$1.IO_L1N_VREF_3; no longer U$2G$2.IO_L09N_3
- net RAMD5: now also U$2G$1.IO_L1P_3; no longer U$2G$2.IO_L10P_3
- net RAMD6: now also U$2G$1.IO_L48P_D7_2; no longer U$2G$2.IO_L04N_2_D6_GCLK13
- net RAMD7: now also U$2G$1.IO_L31P_GCLK31_D14_2; no longer U$2G$2.IO_L05P_2_D4_GCLK14
- net RDY: now also U$2G$1.IO_L2N_3; no longer U$2G$2.IO_31_VREF_3
- net RED: no longer IC6A.G1
- net ROUT: now also U$2G$1.IO_L34N_1; no longer U$2G$2.IO_L08P_1_A2
- net SPISELA/CSO_B: now also U$2G$1.IO_L65N_CSO_B_2; no longer U$2G$2.IO_L01P_2_CSO_B
- net SPISELB: now also U$2G$1.IO_L36N_3; no longer U$2G$2.IO_L08N_3
- net SPISELC: now also U$2G$1.IO_L37P_3; no longer U$2G$2.IO_L08P_3
- net SPI_ACLK: now also U$2G$1.IO_L43N_GCLK22_IRDY2_3; no longer U$2G$2.IO_L05N_3_LHCLK3
- net SPI_AMOSI: now also U$2G$1.IO_L44P_GCLK21_3; no longer U$2G$2.IO_L05P_3_LHCLK2
- net SPI_CLK/CCLK: now also IC8.SCLK, U$12.SCK, U$13.SCK, U$2G$1.IO_L1P_CCLK_2, U$4.SCK, U$9.SCK; no longer U$2G$2.IO_L10N_2_CCLK
- net SPI_IN3: now also U$2G$1.IO_L2P_CMPCLK_2; no longer U$2G$2.IP_69
- net SPI_MISO/DIN: now also U$2G$1.IO_L3P_D0_DIN_MISO_MISO1_2; no longer U$2G$2.IO_L08N_2_DIN_D0
- net SPI_MOSI: now also U$2G$1.IO_L3N_MOSI_CSI_B_MISO0_2; no longer U$2G$2.IO_L02N_2_MOSI_CSI_B
- net SPI_NAUDIO: now also U$2G$1.IO_L64N_SCP4_0; no longer U$2G$2.IO_L02P_0
- net SPI_NFLASH: now also JP10.1
- net SYNC: now also U$2G$1.IO_L62P_0; no longer U$2G$2.IO_L04N_0_GCLK5
- net V12: now also U$2G$2.VCCINT, U$2G$2.VCCINT@1, U$2G$2.VCCINT@2, U$2G$2.VCCINT@3, U$2G$2.VCCINT@4; no longer U$2G$1.VCCINT@0, U$2G$1.VCCINT@1, U$2G$1.VCCINT@2, U$2G$1.VCCINT@3
- net V33: now also C101.1, C104.1, C109.1, C112.1, C121.1, C123.1, C20.1, C28.1, C36.1, C37.1, C64.1, IC6P.VCC, R25.2, U$16.EN, U$2G$2.VCCAUX, U$2G$2.VCCAUX@1, U$2G$2.VCCAUX@2, U$2G$2.VCCAUX@3, U$2G$2.VCCAUX@4, U$2G$2.VCCO_0, U$2G$2.VCCO_0@1, U$2G$2.VCCO_0@2, U$2G$2.VCCO_1, U$2G$2.VCCO_1@1, U$2G$2.VCCO_1@2, U$2G$2.VCCO_2, U$2G$2.VCCO_2@1, U$2G$2.VCCO_3, U$2G$2.VCCO_3@1, U$2G$2.VCCO_3@2, U$7G$2.VCC; no longer U$2G$1.VCCO_0@0, U$2G$1.VCCO_0@1, U$2G$1.VCCO_1@0, U$2G$1.VCCO_1@1, U$2G$1.VCCO_2@0, U$2G$1.VCCO_2@1, U$2G$1.VCCO_2@2, U$2G$1.VCCO_3@0, U$2G$1.VCCO_3@1
- net VCC: no longer C23.2, C63.1, IC6A.A, IC6A.B, IC6P.VCC, QG2.VDD, R23.2, U$17.EN, U$17.VCTRL, U$17.VIN
- net VDA: now also U$2G$1.IO_L42P_GCLK25_TRDY2_3; no longer U$2G$2.IO_L06N_3_LHCLK5
- net VPA: now also U$2G$1.IO_L41P_GCLK27_3; no longer U$2G$2.IO_L07N_3_LHCLK7
- net VPB: now also JP8.1, U$2G$1.IO_L51N_3; no longer U$2G$2.IP_6
- net VSYNC: now also U$2G$1.IO_L34P_1; no longer U$2G$2.IO_L08N_1_A1
Other:
- note added: "/NFLASH (boot) test point"
- note added: "CSA-ULTRACPU-V1.4A-20240206"
- note added: "CSA-ULTRACPU-V2.0A-20240328"
- note added: "CSA-ULTRACPU-V2.0B"
- note added: "CSA-ULTRACPU-V2.0B-20240525"
- note added: "CSA-UTRACPU-V2.0B"
- note added: "For Master SPI config, M[0..1] need to be 01 (M0=1, M1=0) - doing this with '125 when DONE is low M[] are sampled when INIT_B goes high, std I/O after config DONE goes high after initialization is finished. Boot PROM connections: MOSI is SPI MOSI DIN is SPI MISO CSO_B is Boot flash /select CCLK is SPI clock (CCLK is 50 Ohm transmission line - no branches 100/100 termination)"
- note added: "PHI2 test point"
- note added: "Pulling M1 to low for SPI master config on FPGA boot"
- note added: "V1.0B: - Added "Brown Fix" V1.1A: - 3.3/5V level converter - VGA ESD protection diodes V1.4A: - go from RGBI to 6bit RGB (2b/col) (replacing IC6 "brownfix" in the process"
- note added: "V1.1A: - 3.3V/5V level converter V1.2A: - use 74LVC06 instead of HCT - voltage conversion for GRAPHIC V1.2B: - pullup for GRAPHIC V1.3C: - jumper for 3.3V on Bus V2.0A: - remove 16MHz bus signal/oscillator"
- note added: "V1.2A: - Spartan 3E instead of XC95288 V1.2B: - add missing VCCO supply - Pulldown for VSYNC V1.3B: - pull colur handling into FPGA - re-layout - add 70MHz SMD oscillator option - fix FPGA boot, add FPGA boot prom - add /IRQ to FPGA output V1.3C: - move R/-W around to document patch in 1.3B V1.4A: - move from Spartan 3E to Spartan 6 - add option to replace IC6 using FPGA output and IC3 - go from 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"
- note added: "V1.2B: - fix pinout of LDI1117 V1.3B: - adapt C values V1.4A: - fix bypass caps for Spartan 6, RGB V2.0A: - V33 and V12 only, no V25 needed (VCCAUX is 3.3V now)"
- note added: "VPB test point"
- note removed: ""Brown Fix" Changes dark yellow into Brown Used to be included in monitors"
- note removed: "CSA-ULTRACPU-V1.3B-20230811"
- note removed: "CSA-ULTRACPU-V1.3C"
- note removed: "CSA-ULTRACPU-V1.3C-20231117"
- note removed: "CSA-UTRACPU-V1.3C"
- note removed: "For Master SPI config, M[0..2] need to be 001 (M0=1, M1=0, M2=0) - doing this with '125 when DONE is low VS[0..2] select Flash variant M[] and VS[] are sampled when INIT_B goes high, std I/O after config DONE goes high after initialization is finished. Boot PROM connections: MOSI is SPI MOSI DIN is SPI MISO CSO_B is Boot flash /select CCLK is SPI clock (CCLK is 50 Ohm transmission line - no branc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"
- note removed: "V1.0B: - Added "Brown Fix" V1.1A: - 3.3/5V level converter - VGA ESD protection diodes"
- note removed: "V1.1A: - 3.3V/5V level converter V1.2A: - use 74LVC06 instead of HCT - voltage conversion for GRAPHIC V1.2B: - pullup for GRAPHIC V1.3C: - jumper for 3.3V on Bus"
- note removed: "V1.2A: - Spartan 3E instead of XC95288 V1.2B: - add missing VCCO supply - Pulldown for VSYNC V1.3B: - pull colur handling into FPGA - re-layout - add 70MHz SMD oscillator option - fix FPGA boot, add FPGA boot prom - add /IRQ to FPGA output V1.3C: - move R/-W around to document patch in 1.3B"
- note removed: "V1.2B: - fix pinout of LDI1117 V1.3B: - adapt C values"
- moved on the sheet: D1, IC18F, IC19B, IC3A, IC3P, IC7, IC7P, R17, R27, U$7G$2
