File: Board/Audio%2fVideo.kicad_sch (KiCad schematic)
At the start: 10 parts, among them U2 IS61C5128AL-10TLI, X1 SJ1-3513N

Commit message: start r2.2a, moving from VGA to HDMI
Other:
- note added: "CSA-ULTRACPU-V2.2A"
- note removed: "CSA-ULTRACPU-V2.1A"
