File: Board/BUS_I%2fO.kicad_sch (KiCad schematic)
At the start: 14 parts, among them IC13 74244DW, IC14 74LVC14, IC16 74LVC8T245SO24, IC18 74LVC06, IC19 74244DW, IC4 74HCT245DW, IC5 74HCT245DW, P1 CSABUS

Commit message: start r2.2a, moving from VGA to HDMI
Other:
- note added: "CSA-ULTRACPU-V2.2A"
- note removed: "CSA-ULTRACPU-V2.1A"
