File: Board/BUS_I%2fO.kicad_sch (KiCad schematic)
At the start: 14 parts, among them IC13 74244DW, IC14 74LVC14, IC16 74LVC8T245SO24, IC18 74LVC06, IC19 74244DW, IC4 74HCT245DW, IC5 74HCT245DW, P1 CSABUS

Commit message: start working on 3.0 with larger FPGA
Parts:
- added D9: 1N4448, csa_ultracpu:D-5, symbol csa_ultracpu-eagle-import:DIODE-D-5
- added JP1: JP1E, csa_ultracpu:JP1, symbol csa_ultracpu-eagle-import:JP1E
- added R26: 10k, Resistor_SMD:R_0805_2012Metric_Pad1.20x1.40mm_HandSolder, symbol csa_ultracpu-eagle-import:R-EU_0207/2V
Connections:
- net GND: now also R26.1
- net GRAPHIC5V: now also JP1.1
- new net: D9.C, JP1.2, R26.2
- new net PET_VSYNC: D9.A
Other:
- note added: "CSA-ULTRACPU-V3.0A"
- note added: "CSA-ULTRACPU-V3.0A-20260805"
- note added: "Connector to PETIO board for GRAPHIC and VSYNC Interrupt"
- note added: "Protection against accidently connecting the wrong way around (Note: prevents O.C. receiver logic)"
- note added: "V1.1A: - 3.3V/5V level converter V1.2A: - use 74LVC06 instead of HCT - voltage conversion for GRAPHIC V1.2B: - pullup for GRAPHIC V1.3C: - jumper for 3.3V on Bus V2.0A: - remove 16MHz bus signal/oscillator V2.1A: - fix Kicad import wiring bug (where FA16,17,18 were connected) V3.0A: - move Graphics and PET_VSYNC handling to this page"
- note removed: "CSA-ULTRACPU-V2.1A-20241207"
- note removed: "CSA-ULTRACPU-V2.2A"
- note removed: "V1.1A: - 3.3V/5V level converter V1.2A: - use 74LVC06 instead of HCT - voltage conversion for GRAPHIC V1.2B: - pullup for GRAPHIC V1.3C: - jumper for 3.3V on Bus V2.0A: - remove 16MHz bus signal/oscillator V2.1A: - fix Kicad import wiring bug (where FA16,17,18 were connected)"
- moved on the sheet: IC13C, IC14G, IC18F, IC18G, IC19C, IC4B, IC5B, R27

Commit message: more layout work
Connections:
- net A12 renamed FA12
- net A13 renamed FA13
- net A14 renamed FA14
- net A15 renamed FA15
Other:
- note added: "CSA-ULTRACPU-V3.0A-20260905"
- note added: "V1.1A: - 3.3V/5V level converter V1.2A: - use 74LVC06 instead of HCT - voltage conversion for GRAPHIC V1.2B: - pullup for GRAPHIC V1.3C: - jumper for 3.3V on Bus V2.0A: - remove 16MHz bus signal/oscillator V2.1A: - fix Kicad import wiring bug (where FA16,17,18 were connected) V3.0A: - move Graphics and PET_VSYNC handling to this page - use new FA12-FA15 on bus out"
- note removed: "CSA-ULTRACPU-V3.0A-20260805"
- note removed: "V1.1A: - 3.3V/5V level converter V1.2A: - use 74LVC06 instead of HCT - voltage conversion for GRAPHIC V1.2B: - pullup for GRAPHIC V1.3C: - jumper for 3.3V on Bus V2.0A: - remove 16MHz bus signal/oscillator V2.1A: - fix Kicad import wiring bug (where FA16,17,18 were connected) V3.0A: - move Graphics and PET_VSYNC handling to this page"

Commit message: more layout work
Parts:
- D9: footprint csa_ultracpu:D-5 -> Diode_SMD:D_SOD-123; LCSC (none) -> C2128
- JP1: footprint csa_ultracpu:JP1 -> Connector_PinHeader_2.54mm:PinHeader_1x02_P2.54mm_Horizontal
Connections:
- net PET_VSYNC: now also D9.2 (A); no longer D9.A
- net at JP1.2, R26.2: now also D9.1 (C); no longer D9.C
Changed lines of the file:
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@@
 			)
 		)
-		(property "Footprint" "csa_ultracpu:JP1"
+		(property "Footprint" "Connector_PinHeader_2.54mm:PinHeader_1x02_P2.54mm_Horizontal"
 			(at 327.66 149.86 0)
 			(hide yes)
@@
 			)
 		)
-		(property "Footprint" "csa_ultracpu:D-5"
+		(property "Footprint" "Diode_SMD:D_SOD-123"
 			(at 307.34 160.02 0)
 			(hide yes)
@@
 			)
 		)
-		(pin "A"
-		)
-		(pin "C"
-		)
-		(instances
+		(property "LCSC" "C2128"
+			(at 307.34 160.02 0)
+			(hide yes)
+			(show_name no)
+			(do_not_autoplace no)
+			(effects
+				(font
+					(size 1.27 1.27)
+				)
+			)
+		)
+		(pin "1"
+		)
+		(pin "2"
+		)
+		(instances

Commit message: more layout work
Other:
- note added: "V2.0A: - remove 16MHz bus signal/oscillator V2.1A: - fix Kicad import wiring bug (where FA16,17,18 were connected) V3.0A: - move Graphics and PET_VSYNC handling to this page - use new FA12-FA15 on bus out"
- note removed: "V1.1A: - 3.3V/5V level converter V1.2A: - use 74LVC06 instead of HCT - voltage conversion for GRAPHIC V1.2B: - pullup for GRAPHIC V1.3C: - jumper for 3.3V on Bus V2.0A: - remove 16MHz bus signal/oscillator V2.1A: - fix Kicad import wiring bug (where FA16,17,18 were connected) V3.0A: - move Graphics and PET_VSYNC handling to this page - use new FA12-FA15 on bus out"
Changed lines of the file:
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@@
 		)
 	)
-	(text "V1.1A:\n- 3.3V/5V level converter\nV1.2A:\n- use 74LVC06 instead of HCT\n- voltage conversion for GRAPHIC\nV1.2B:\n- pullup for GRAPHIC\nV1.3C:\n- jumper for 3.3V on Bus\nV2.0A:\n- remove 16MHz bus signal/oscillator\nV2.1A:\n- fix Kicad import wiring bug (where FA16,17,18 were connected)\nV3.0A:\n- move Graphics and PET_VSYNC handling to this page\n- use new FA12-FA15 on bus out"
+	(text "V2.0A:\n- remove 16MHz bus signal/oscillator\nV2.1A:\n- fix Kicad import wiring bug (where FA16,17,18 were connected)\nV3.0A:\n- move Graphics and PET_VSYNC handling to this page\n- use new FA12-FA15 on bus out"
 		(exclude_from_sim no)
 		(at 231.14 323.85 0)

Commit message: layout done
Parts:
- IC13, IC19: LCSC (none) -> C6776
- IC14: LCSC (none) -> C133541
- IC16: LCSC (none) -> C2677625
- IC18: LCSC (none) -> C7658
- IC4, IC5: LCSC (none) -> C132267
- JP1: LCSC (none) -> C54570432
- JP6: LCSC (none) -> C234182
- P1: LCSC (none) -> C5173362
- R16, R17, R26, R27, R6: LCSC (none) -> C17414
- RN2: LCSC (none) -> C8692
