File: Board/BUS_I%2fO.kicad_sch (KiCad schematic)
At the start: 17 parts, among them IC13 74244DW, IC14 74LVC14, IC16 74LVC8T245SO24, IC18 74LVC06, IC19 74244DW, IC4 74HCT245DW, IC5 74HCT245DW, P1 CSABUS

Commit message: fix diode footprint in bom
Parts:
- D9: LCSC C2128 -> C81598
Changed lines of the file:
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@@
 			)
 		)
-		(property "LCSC" "C2128"
+		(property "LCSC" "C81598"
 			(at 307.34 160.02 0)
 			(hide yes)
