File: Board/USB.kicad_sch (KiCad schematic)
At the start: 29 parts, among them IC8 MAX3421E, Q2 32kHz, Q3 12MHz

Commit message: more work on r2.1a - only bom xls is missing/outdated
Parts:
- C9: value 1.0u Cer -> 1u
Changed lines of the file:
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@@
 			)
 		)
-		(property "Value" "1.0u Cer"
+		(property "Value" "1u"
 			(at 136.144 157.099 0)
 			(effects

Commit message: start r2.2a, moving from VGA to HDMI
Parts:
- removed JP3: JP1E, csa_ultracpu:JP1, symbol csa_ultracpu-eagle-import:JP1E
- added JP15: JP2E, csa_ultracpu:JP2, symbol csa_ultracpu-eagle-import:JP2E
Connections:
- net VBUF: now also JP15.1
- net at JP2.1, U$13.3 (VBAT): now also JP15.2
- new net VBATT: JP15.3
Other:
- note added: "CSA-ULTRACPU-V2.2A"
- note added: "CSA-ULTRACPU-V2.2A-20260602"
- note added: "JP15 to use RTC Power 1-2: from CSA BUS 2-3: from CR2032 open: ext. pwr (JP2)"
- note added: "V1.1A: - added USB ESD protection diodes V2.1A: - replaced non-commercial footprint for USB chip - added boot option jumpers on USB GPIN V2.2A: - add CR2032 battery power option"
- note removed: "CSA-ULTRACPU-V2.1A"
- note removed: "CSA-ULTRACPU-V2.1A-20241207"
- note removed: "JP3 to use VBUF from CSA BUS"
- note removed: "V1.1A: - added USB ESD protection diodes V2.1A: - replaced non-commercial footprint for USB chip - added boot option jumpers on USB GPIN"
Changed lines of the file:
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@@
 (kicad_sch
-	(version 20231120)
+	(version 20250114)
 	(generator "eeschema")
-	(generator_version "8.0")
+	(generator_version "9.0")
 	(paper "User" 334.823 218.592)
+	(text "CSA-ULTRACPU-V2.2A"
+		(exclude_from_sim no)
+		(at 208.28 167.64 0)
+		(effects
+			(font
+				(size 3.81 3.2385)
+			)
+			(justify left bottom)
+		)
+	)
+	(text "V1.1A:\n- added USB ESD protection diodes\nV2.1A:\n- replaced non-commercial footprint for USB chip\n- added boot option jumpers on USB GPIN\nV2.2A:\n- add CR2032 battery power option"
+		(exclude_from_sim no)
+		(at 115.57 194.31 0)
+		(effects
+			(font
+				(size 2.54 2.159)
+			)
+			(justify left bottom)
+		)
+	)
+	(text "CSA-ULTRACPU-V2.2A-20260602"
+		(exclude_from_sim no)
+		(at 208.28 190.5 0)
+		(effects
+			(font
+				(size 2.54 2.159)
+			)
+			(justify left bottom)
+		)
+	)
+	(text "(C) A. Fachat"
+		(exclude_from_sim no)
+		(at 208.28 172.72 0)
+		(effects
+			(font
+				(size 2.54 2.159)
+			)
+			(justify left bottom)
+		)
+	)
+	(text "Connect Coin Cell\non JP2"
+		(exclude_from_sim no)
+		(at 267.97 68.58 0)
+		(effects
+			(font
+				(size 2.54 2.159)
+			)
+			(justify left bottom)
+		)
+	)
+	(text "Watch orientation on board~{}"
+		(exclude_from_sim no)
+		(at 66.04 162.56 0)
+		(effects
+			(font
+				(size 2.54 2.159)
+			)
+			(justify left bottom)
+		)
+	)
+	(text "JP15 to use RTC Power\n1-2: from CSA BUS\n2-3: from CR2032\nopen: ext. pwr (JP2)"
+		(exclude_from_sim no)
+		(at 266.7 36.83 0)
+		(effects
+			(font
+				(size 2.54 2.159)
+			)
+			(justify left bottom)
+		)
+	)
 	(junction
 		(at 241.3 35.56)
@@
 	(wire
 		(pts
+			(xy 283.21 45.72) (xy 287.02 45.72)
+		)
+		(stroke
+			(width 0)
+			(type default)
+		)
+	)
+	(wire
+		(pts
 			(xy 228.6 53.34) (xy 237.49 53.34)
 		)
@@
 	(wire
 		(pts
+			(xy 271.78 57.15) (xy 287.02 57.15)
+		)
+		(stroke
+			(width 0.1524)
+			(type solid)
+		)
+	)
+	(wire
+		(pts
 			(xy 116.84 104.14) (xy 132.08 104.14)
 		)
@@
 	(wire
 		(pts
+			(xy 283.21 50.8) (xy 283.21 45.72)
+		)
+		(stroke
+			(width 0)
+			(type default)
+		)
+	)
+	(wire
+		(pts
 			(xy 152.4 142.24) (xy 152.4 139.7)
 		)
@@
 	(wire
 		(pts
-			(xy 284.48 50.8) (xy 271.78 50.8)
-		)
-		(stroke
-			(width 0.1524)
-			(type solid)
-		)
-	)
-	(wire
-		(pts
 			(xy 261.62 66.04) (xy 261.62 58.42)
 		)
@@
 	(wire
 		(pts
-			(xy 271.78 48.26) (xy 271.78 50.8)
+			(xy 271.78 48.26) (xy 271.78 57.15)
 		)
 		(stroke
@@
 	(wire
 		(pts
-			(xy 269.24 50.8) (xy 269.24 48.26)
+			(xy 274.32 50.8) (xy 274.32 48.26)
 		)
 		(stroke
@@
 	(wire
 		(pts
-			(xy 261.62 50.8) (xy 269.24 50.8)
+			(xy 261.62 50.8) (xy 274.32 50.8)
 		)
 		(stroke
@@
 	(wire
 		(pts
+			(xy 276.86 48.26) (xy 276.86 50.8)
+		)
+		(stroke
+			(width 0)
+			(type default)
+		)
+	)
+	(wire
+		(pts
 			(xy 132.08 53.34) (xy 63.5 53.34)
 		)
@@
 	(wire
 		(pts
+			(xy 276.86 50.8) (xy 283.21 50.8)
+		)
+		(stroke
+			(width 0)
+			(type default)
+		)
+	)
+	(wire
+		(pts
 			(xy 116.84 149.86) (xy 121.92 149.86)
 		)
@@
 		)
 	)
-	(text "CSA-ULTRACPU-V2.1A"
-		(exclude_from_sim no)
-		(at 208.28 167.64 0)
-		(effects
-			(font
-				(size 3.81 3.2385)
-			)
-			(justify left bottom)
-		)
-	)
-	(text "V1.1A:\n- added USB ESD protection diodes\nV2.1A:\n- replaced non-commercial footprint for USB chip\n- added boot option jumpers on USB GPIN"
-		(exclude_from_sim no)
-		(at 108.712 190.754 0)
-		(effects
-			(font
-				(size 2.54 2.159)
-			)
-			(justify left bottom)
-		)
-	)
-	(text "CSA-ULTRACPU-V2.1A-20241207"
-		(exclude_from_sim no)
-		(at 208.28 190.5 0)
-		(effects
-			(font
-				(size 2.54 2.159)
-			)
-			(justify left bottom)
-		)
-	)
-	(text "(C) A. Fachat"
-		(exclude_from_sim no)
-		(at 208.28 172.72 0)
-		(effects
-			(font
-				(size 2.54 2.159)
-			)
-			(justify left bottom)
-		)
-	)
-	(text "Connect Coin Cell\non JP2"
-		(exclude_from_sim no)
-		(at 271.78 60.96 0)
-		(effects
-			(font
-				(size 2.54 2.159)
-			)
-			(justify left bottom)
-		)
-	)
-	(text "Watch orientation on board~{}"
-		(exclude_from_sim no)
-		(at 66.04 162.56 0)
-		(effects
-			(font
-				(size 2.54 2.159)
-			)
-			(justify left bottom)
-		)
-	)
-	(text "JP3 to use VBUF\nfrom CSA BUS"
-		(exclude_from_sim no)
-		(at 271.78 38.1 0)
-		(effects
-			(font
-				(size 2.54 2.159)
-			)
-			(justify left bottom)
-		)
-	)
 	(label "/USBINT"
 		(at 48.26 106.68 0)
-		(fields_autoplaced yes)
 		(effects
 			(font
@@
 	(label "DETECT"
 		(at 76.2 78.74 0)
-		(fields_autoplaced yes)
 		(effects
 			(font
@@
 	)
 	(global_label "VBUF"
-		(shape bidirectional)
-		(at 276.86 50.8 0)
+		(shape input)
+		(at 287.02 57.15 0)
 		(fields_autoplaced yes)
 		(effects
@@
 		)
 		(property "Intersheetrefs" "${INTERSHEET_REFS}"
-			(at 285.5563 50.8 0)
+			(at 294.6273 57.15 0)
 			(effects
 				(font
@@
 		)
 	)
+	(global_label "VBATT"
+		(shape input)
+		(at 287.02 45.72 0)
+		(fields_autoplaced yes)
+		(effects
+			(font
+				(size 1.2446 1.2446)
+			)
+			(justify left)
+		)
+		(property "Intersheetrefs" "${INTERSHEET_REFS}"
+			(at 295.22 45.72 0)
+			(effects
+				(font
+					(size 1.27 1.27)
+				)
+				(justify left)
+				(hide yes)
+			)
+		)
+	)
 	(global_label "/IRQ"
 		(shape bidirectional)
@@
 	)
 	(symbol
-		(lib_id "csa_ultracpu-eagle-import:JP1E")
-		(at 269.24 45.72 0)
-		(unit 1)
-		(exclude_from_sim no)
-		(in_bom yes)
-		(on_board yes)
-		(dnp no)
-		(property "Reference" "JP3"
-			(at 267.97 45.72 90)
-			(effects
-				(font
-					(size 1.778 1.5113)
-				)
-				(justify left bottom)
-			)
-		)
-		(property "Value" "JP1E"
-			(at 274.955 45.72 90)
-			(effects
-				(font
-					(size 1.778 1.5113)
-				)
-				(justify left bottom)
-				(hide yes)
-			)
-		)
-		(property "Footprint" "csa_ultracpu:JP1"
-			(at 269.24 45.72 0)
-			(effects
-				(font
-					(size 1.27 1.27)
-				)
-				(hide yes)
-			)
-		)
-		(property "Datasheet" ""
-			(at 269.24 45.72 0)
-			(effects
-				(font
-					(size 1.27 1.27)
-				)
-				(hide yes)
-			)
-		)
-		(property "Description" ""
-			(at 269.24 45.72 0)
-			(effects
-				(font
-					(size 1.27 1.27)
-				)
-				(hide yes)
-			)
-		)
-		(pin "1"
-		)
-		(pin "2"
-		)
-		(instances
-			(project ""
-				(path "/381336a5-a662-4c84-a650-90475fa59a97/2002a839-3bb0-44ee-a1e7-391421f825e7"
-					(reference "JP3")
-					(unit 1)
-				)
-			)
-		)
-	)
-	(symbol
 		(lib_id "csa_ultracpu-eagle-import:GND")
 		(at 137.16 129.54 0)
@@
 					(unit 1)
 				)
+			)
+		)
+	)
+	(symbol
+		(lib_id "csa_ultracpu-eagle-import:JP2E")
+		(at 274.32 45.72 0)
+		(unit 1)
+		(exclude_from_sim no)
+		(in_bom yes)
+		(on_board yes)
+		(dnp no)
+		(property "Reference" "JP15"
+			(at 270.51 45.72 90)
+			(effects
+				(font
+					(size 1.778 1.5113)
+				)
+				(justify left bottom)
+			)
+		)
+		(property "Value" "JP2E"
+			(at 280.035 45.72 90)
+			(effects
+				(font
+					(size 1.778 1.5113)
+				)
+				(justify left bottom)
+				(hide yes)
+			)
+		)
+		(property "Footprint" "csa_ultracpu:JP2"
+			(at 274.32 45.72 0)
+			(effects
+				(font
+					(size 1.27 1.27)
+				)
+				(hide yes)
+			)
+		)
+		(property "Datasheet" ""
+			(at 274.32 45.72 0)
+			(effects
+				(font
+					(size 1.27 1.27)
+				)
+				(hide yes)
+			)
+		)
+		(property "Description" ""
+			(at 274.32 45.72 0)
+			(effects
+				(font
+					(size 1.27 1.27)
+				)
+				(hide yes)
+			)
+		)
+		(pin "1"
+		)
+		(pin "2"
+		)
+		(pin "3"
+		)
+		(instances
+			(project "csa_ultracpu"
+				(path "/381336a5-a662-4c84-a650-90475fa59a97/2002a839-3bb0-44ee-a1e7-391421f825e7"
+					(reference "JP15")
+					(unit 1)
+				)
