File: Board/USB.kicad_sch (KiCad schematic)
At the start: 29 parts, among them IC8 MAX3421E, Q2 32kHz, Q3 12MHz

Commit message: more layout work
Other:
- note added: "CSA-ULTRACPU-V3.0A"
- note removed: "CSA-ULTRACPU-V2.2A"
Changed lines of the file:
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@@
 	(generator_version "10.0")
 	(paper "User" 334.823 218.592)
-	(text "CSA-ULTRACPU-V2.2A"
+	(text "CSA-ULTRACPU-V3.0A"
 		(exclude_from_sim no)
 		(at 208.28 167.64 0)

Commit message: layout done
Parts:
- added C73: 100n, Capacitor_SMD:C_0603_1608Metric_Pad1.08x0.95mm_HandSolder, symbol Device:C
- added C74: 22u, csa_ultracpu:C0805, symbol csa_ultracpu-eagle-import:C-EUC0805
- added J2: Micro_SD_Card_Det2, Connector_Card:microSD_HC_Molex_104031-0811, symbol Connector:Micro_SD_Card_Det2
- added U2: 74LVC125, Package_SO:SO-14_3.9x8.65mm_P1.27mm, symbol 74xx:74LVC125
- C16, C21, C27: LCSC (none) -> C14663
- C29, C30, C39, C40: LCSC (none) -> C1647
- C9: LCSC (none) -> C15849
- D5, D6, D8: LCSC (none) -> C402212
- IC8: LCSC (none) -> C2651881
- JP12, JP13, JP2: LCSC (none) -> C234182
- JP15: LCSC (none) -> C587036
- Q2: LCSC (none) -> C3013591
- Q3: LCSC (none) -> C16369
- R1, R2, R4: LCSC (none) -> C17634
- R12, R5: LCSC (none) -> C17414
- U$12: LCSC (none) -> C27438
- U$13: LCSC (none) -> C627708
- U$14, U$15: LCSC (none) -> C2687118
- USB1: LCSC (none) -> C456018
Connections:
- net GND: now also C73.2, C74.2, J2.6 (VSS), J2.SH (SHIELD), U2.7 (GND)
- net SPI_CLK/CCLK: now also U2.5
- net SPI_IN3: now also U2.8; no longer U$12.DO
- net SPI_MOSI: now also U2.2
- net SPI_NSEL3: now also U2.1, U2.10, U2.12, U2.13, U2.4
- net V33: now also C73.1, C74.1, J2.4 (VDD), U2.14 (VCC)
- new net: J2.7 (DAT0), U$12.DO, U2.9
- new net: J2.2 (DAT3/CD), U2.11
- new net: J2.3 (CMD), U2.3
- new net: J2.5 (CLK), U2.6
Other:
- moved on the sheet: C16, C21, C27, C29, C30, C39, C40, C9, D5, D6, D8, IC8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

Commit message: as submitted
Parts:
- IC8: footprint Package_QFP:LQFP-32_5x5mm_P0.5mm -> Package_DFN_QFN:VQFN-32-1EP_5x5mm_P0.5mm_EP3.15x3.15mm; LCSC C2651881 -> C1870151
Changed lines of the file:
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@@
 			)
 		)
-		(property "Footprint" "Package_QFP:LQFP-32_5x5mm_P0.5mm"
+		(property "Footprint" "Package_DFN_QFN:VQFN-32-1EP_5x5mm_P0.5mm_EP3.15x3.15mm"
 			(at 117.475 177.165 0)
 			(hide yes)
@@
 			)
 		)
-		(property "LCSC" "C2651881"
+		(property "LCSC" "C1870151"
 			(at 102.235 154.305 0)
 			(hide yes)
