File: Board/CPU,RAM,ROM.kicad_sch (KiCad schematic)
At the start: 25 parts, among them IC3 74LVC125, IC6 741G04DBV, IC7 74LVC138, U1 IS61C5128AL-10TLI, X3 SG-8002CE

Commit message: update
Connections:
- net /RAMWE: now also U$2.93 (IO_L41P_GCLK9_IRDY1_1); no longer U$2.55 (IO_L30N_GCLK0_USERCCLK_2)
- net A1: now also U$2.46 (IO_L49P_D3_2); no longer U$2.56 (IO_L30P_GCLK1_D13_2)
- net HDMI-CK+: now also U$2.48 (IO_L48P_D7_2); no longer U$2.93 (IO_L41P_GCLK9_IRDY1_1)
- net HDMI-CK-: now also U$2.47 (IO_L48N_RDRW_B_VREF_2); no longer U$2.92 (IO_L41N_GCLK8_1)
- net HDMI-D0+: now also U$2.51 (IO_L31P_GCLK31_D14_2); no longer U$2.95 (IO_L40P_GCLK11_1)
- net HDMI-D0-: now also U$2.50 (IO_L31N_GCLK30_D15_2); no longer U$2.94 (IO_L40N_GCLK10_1)
- net HDMI-D1+: now also U$2.56 (IO_L30P_GCLK1_D13_2); no longer U$2.98 (IO_L34P_1)
- net HDMI-D1-: now also U$2.55 (IO_L30N_GCLK0_USERCCLK_2); no longer U$2.97 (IO_L34N_1)
- net HDMI-D2+: now also U$2.58 (IO_L14P_D11_2); no longer U$2.100 (IO_L33P_1)
- net HDMI-D2-: now also U$2.57 (IO_L14N_D12_2); no longer U$2.99 (IO_L33N_1)
- net RAMA12: now also U$2.100 (IO_L33P_1); no longer U$2.47 (IO_L48N_RDRW_B_VREF_2)
- net RAMA13: now also U$2.99 (IO_L33N_1); no longer U$2.50 (IO_L31N_GCLK30_D15_2)
- net RAMA5: now also U$2.94 (IO_L40N_GCLK10_1); no longer U$2.51 (IO_L31P_GCLK31_D14_2)
- net RAMA6: now also U$2.95 (IO_L40P_GCLK11_1); no longer U$2.48 (IO_L48P_D7_2)
- net RAMA7: now also U$2.97 (IO_L34N_1); no longer U$2.46 (IO_L49P_D3_2)
- net RAMD3: now also U$2.92 (IO_L41N_GCLK8_1); no longer U$2.57 (IO_L14N_D12_2)
- net RAMD4: now also U$2.98 (IO_L34P_1); no longer U$2.58 (IO_L14P_D11_2)

Commit message: start working on 3.0 with larger FPGA
Parts:
- removed D9: 1N4448, csa_ultracpu:D-5, symbol csa_ultracpu-eagle-import:DIODE-D-5
- removed unit 2 of IC3
- removed unit 1 of IC3
- removed unit 1 of IC7
- removed JP1, JP4: JP1E, csa_ultracpu:JP1, symbol csa_ultracpu-eagle-import:JP1E
- removed R25, R26: 10k, Resistor_SMD:R_0805_2012Metric_Pad1.20x1.40mm_HandSolder, symbol csa_ultracpu-eagle-import:R-EU_0207/2V
- removed R29: 330, csa_ultracpu:0207_2V, symbol csa_ultracpu-eagle-import:R-EU_0207/2V
- removed U$2: XC6SLX9-TQG144, csa_ultracpu:TQFP144, symbol csa_ultracpu-eagle-import:XC9SLX9-TQG144
- removed unit 2 of U$7
- removed unit 1 of U$7
- removed U1: IS61C5128AL-10TLI, Package_SO:TSOP-II-44_10.16x18.41mm_P0.8mm, symbol Memory_RAM:IS61C5128AL-10TLI
- added U1: IS61WV51216EDALL, Package_SO:TSOP-II-44_10.16x18.41mm_P0.8mm, symbol csa_ultracpu-eagle-import:IS61WV51216EDALL
Connections:
- net A0: now also U1.1 (A0)
- net A1: now also U1.2 (A1)
- net A10: now also U1.23 (A10)
- net A11: now also U1.24 (A11)
- net A2: now also U1.3 (A2)
- net A3: now also U1.4 (A3)
- net A4: now also U1.5 (A4)
- net A5: now also U1.18 (A5)
- net A6: now also U1.19 (A6)
- net A7: now also U1.20 (A7)
- net A8: now also U1.21 (A8)
- net A9: now also U1.22 (A9)
- net D0: now also U1.29 (I/O8), U1.7 (I/O0)
- net D1: now also U1.30 (I/O9), U1.8 (I/O1)
- net D2: now also U1.31 (I/O10), U1.9 (I/O2)
- net D3: now also U1.10 (I/O3), U1.32 (I/O11)
- net D4: now also U1.13 (I/O4), U1.35 (I/O12)
- net D5: now also U1.14 (I/O5), U1.36 (I/O13)
- net D6: now also U1.15 (I/O6), U1.37 (I/O14)
- net D7: now also U1.16 (I/O7), U1.38 (I/O15)
- net FA15: now also U1.42 (A15)
- net FA16: now also U1.43 (A16)
- net FA17: now also U1.44 (A17)
- net FA18: now also U1.28 (A18)
- net GND: now also U1.12 (GND), U1.34 (GND)
- net R/-W: now also U1.17 (~{WE})
- net V33: now also U1.11 (VDD), U1.33 (VDD)
- net /FRAMSEL: now also U1.41 (~{OE}), U1.6 (~{CE})
- net 50M renamed QCLK
- new net FA12: U1.25 (A12)
- new net FA13: U1.26 (A13)
- new net FA14: U1.27 (A14)
- new net /FRAMLB: U1.39 (~{LB})
- new net /FRAMUB: U1.40 (~{UB})
Other:
- note added: "CSA-UTRACPU-V3.0A"
- note added: "Fast RAM"
- note added: "V2.0A: - use CCLK for all SPI clocks - add switchable CPU BE input - VCCAUX is 3.3V now - Added test points V2.0B: - IC6 power supply to 3.3V instead of 5V - Pulldown /RES as long as DONE is low V2.1A: - use TSOP-II 44 pin package for SRAM - use 3225 package for 54MHz SMD oscillator V3.0A: - go from VGA to HDMI - go to larger FPGA in BGA package, move FPGA to own page - use 16bit Fast RAM IC"
- note removed: "CSA-UTRACPU-V2.2A"
- note removed: "For Master SPI config, M[0..1] need to be 01 (M0=1, M1=0) - doing this with '125 when DONE is low M[] are sampled when INIT_B goes high, std I/O after config DONE goes high after initialization is finished. Boot PROM connections: MOSI is SPI MOSI DIN is SPI MISO CSO_B is Boot flash /select CCLK is SPI clock (CCLK is 50 Ohm transmission line - no branches 100/100 termination)"
- note removed: "HSWAP pulldown during configuration to enable pullups on config+I/O pins"
- note removed: "Protection against accidently connecting the wrong way around"
- note removed: "Pulling M1 to low for SPI master config on FPGA boot"
- note removed: "V2.0A: - use CCLK for all SPI clocks - add switchable CPU BE input - VCCAUX is 3.3V now - Added test points V2.0B: - IC6 power supply to 3.3V instead of 5V - Pulldown /RES as long as DONE is low V2.1A: - use TSOP-II 44 pin package for SRAM - use 3225 package for 54MHz SMD oscillator V2.2A: - go from VGA to HDMI"
- moved on the sheet: IC3C, IC3E, IC6A, IC6B, IC7B, JP10, JP11, JP7, JP8, JP9, R10, R11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

Commit message: layout work
Parts:
- removed unit 3 of U$1
- removed U$7: XILINXPROG, csa_ultracpu:FLAT10BOX, symbol csa_ultracpu-eagle-import:XILINXPROG
- renumbered IC3 to IC1
Connections:
- net D0: now also U1.38 (I/O15); no longer U1.29 (I/O8)
- net D1: now also U1.37 (I/O14); no longer U1.30 (I/O9)
- net D2: now also U1.36 (I/O13); no longer U1.31 (I/O10)
- net D3: now also U1.35 (I/O12); no longer U1.32 (I/O11)
- net D4: now also U1.32 (I/O11); no longer U1.35 (I/O12)
- net D5: now also U1.31 (I/O10); no longer U1.36 (I/O13)
- net D6: now also U1.30 (I/O9); no longer U1.37 (I/O14)
- net D7: now also U1.29 (I/O8); no longer U1.38 (I/O15)

Commit message: layout work
Connections:
- net SPI_MISO/DIN: no longer U$4.2 (SO)
- net /FPGA_BOOT renamed /FPGA_BOOT
- net SPI_NFLASH renamed /SPI_FLASH
Changed lines of the file:
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@@
 	)
 	(junction
+		(at 90.17 83.82)
+		(diameter 0)
+		(color 0 0 0 0)
+	)
+	(junction
 		(at 224.79 184.15)
 		(diameter 0)
@@
 	)
 	(junction
+		(at 90.17 40.64)
+		(diameter 0)
+		(color 0 0 0 0)
+	)
+	(junction
 		(at 181.61 207.01)
 		(diameter 0)
@@
 	)
 	(junction
+		(at 95.25 45.72)
+		(diameter 0)
+		(color 0 0 0 0)
+	)
+	(junction
 		(at 52.705 212.09)
 		(diameter 0)
@@
 	)
 	(junction
-		(at 95.25 76.2)
-		(diameter 0)
-		(color 0 0 0 0)
-	)
-	(junction
 		(at 353.06 74.93)
 		(diameter 0)
@@
 	)
 	(junction
-		(at 97.79 81.28)
-		(diameter 0)
-		(color 0 0 0 0)
-	)
-	(junction
 		(at 256.54 72.39)
 		(diameter 0)
@@
 	)
 	(junction
-		(at 90.17 83.82)
-		(diameter 0)
-		(color 0 0 0 0)
-	)
-	(junction
 		(at 229.87 148.59)
 		(diameter 0)
@@
 		(color 0 0 0 0)
 	)
-	(junction
-		(at 92.71 78.74)
-		(diameter 0)
-		(color 0 0 0 0)
-	)
 	(wire
 		(pts
@@
 	(wire
 		(pts
-			(xy 72.39 81.28) (xy 97.79 81.28)
+			(xy 72.39 81.28) (xy 95.25 81.28)
 		)
 		(stroke
@@
 	(wire
 		(pts
+			(xy 95.25 45.72) (xy 107.95 45.72)
+		)
+		(stroke
+			(width 0.1524)
+			(type solid)
+		)
+	)
+	(wire
+		(pts
 			(xy 214.63 163.83) (xy 224.79 163.83)
 		)
@@
 	(wire
 		(pts
-			(xy 72.39 43.18) (xy 92.71 43.18)
+			(xy 72.39 43.18) (xy 107.95 43.18)
 		)
 		(stroke
@@
 	(wire
 		(pts
-			(xy 72.39 76.2) (xy 95.25 76.2)
+			(xy 72.39 76.2) (xy 90.17 76.2)
 		)
 		(stroke
@@
 	(wire
 		(pts
-			(xy 92.71 78.74) (xy 115.57 78.74)
-		)
-		(stroke
-			(width 0.1524)
-			(type solid)
-		)
-	)
-	(wire
-		(pts
 			(xy 46.99 181.61) (xy 55.88 181.61)
 		)
@@
 	(wire
 		(pts
-			(xy 97.79 81.28) (xy 97.79 45.72)
+			(xy 95.25 81.28) (xy 95.25 45.72)
 		)
 		(stroke
@@
 	(wire
 		(pts
-			(xy 72.39 40.64) (xy 95.25 40.64)
+			(xy 72.39 40.64) (xy 90.17 40.64)
 		)
 		(stroke
@@
 	(wire
 		(pts
+			(xy 90.17 40.64) (xy 107.95 40.64)
+		)
+		(stroke
+			(width 0.1524)
+			(type solid)
+		)
+	)
+	(wire
+		(pts
 			(xy 232.41 194.31) (xy 217.17 194.31)
 		)
@@
 	(wire
 		(pts
-			(xy 95.25 40.64) (xy 95.25 76.2)
+			(xy 90.17 40.64) (xy 90.17 76.2)
 		)
 		(stroke
@@
 	(wire
 		(pts
-			(xy 97.79 81.28) (xy 113.03 81.28)
-		)
-		(stroke
-			(width 0.1524)
-			(type solid)
-		)
-	)
-	(wire
-		(pts
 			(xy 86.36 173.99) (xy 92.71 173.99)
 		)
@@
 	(wire
 		(pts
-			(xy 72.39 45.72) (xy 97.79 45.72)
+			(xy 72.39 45.72) (xy 95.25 45.72)
 		)
 		(stroke
@@
 	(wire
 		(pts
-			(xy 90.17 83.82) (xy 113.03 83.82)
+			(xy 90.17 83.82) (xy 109.22 83.82)
 		)
 		(stroke
@@
 	(wire
 		(pts
-			(xy 95.25 76.2) (xy 115.57 76.2)
-		)
-		(stroke
-			(width 0.1524)
-			(type solid)
-		)
-	)
-	(wire
-		(pts
 			(xy 86.36 171.45) (xy 93.98 171.45)
 		)
@@
 		)
 	)
-	(label "SPI_NFLASH"
-		(at 77.47 83.82 0)
-		(effects
-			(font
-				(size 0.889 0.889)
-			)
-			(justify left bottom)
-		)
-	)
 	(label "VPB"
 		(at 219.71 148.59 0)
@@
 		)
 	)
-	(label "/FPGA_BOOT"
-		(at 74.93 48.26 0)
-		(effects
-			(font
-				(size 1.2446 1.2446)
-			)
-			(justify left bottom)
-		)
-	)
 	(global_label "A8"
 		(shape input)
@@
 		)
 	)
+	(global_label "{slash}FPGA_BOOT"
+		(shape bidirectional)
+		(at 107.95 48.26 0)
+		(fields_autoplaced yes)
+		(effects
+			(font
+				(size 1.2446 1.2446)
+			)
+			(justify left)
+		)
+		(property "Intersheetrefs" "${INTERSHEET_REFS}"
+			(at 123.6399 48.26 0)
+			(hide yes)
+			(show_name no)
+			(do_not_autoplace no)
+			(effects
+				(font
+					(size 1.27 1.27)
+				)
+				(justify left)
+			)
+		)
+	)
 	(global_label "SPI_MOSI"
 		(shape bidirectional)
-		(at 74.93 40.64 0)
+		(at 107.95 40.64 0)
 		(fields_autoplaced yes)
 		(effects
@@
 		)
 		(property "Intersheetrefs" "${INTERSHEET_REFS}"
-			(at 87.4194 40.64 0)
+			(at 120.4394 40.64 0)
 			(hide yes)
 			(show_name no)
@@
 	(global_label "SPI_MISO/DIN"
 		(shape bidirectional)
-		(at 74.93 43.18 0)
+		(at 107.95 43.18 0)
 		(fields_autoplaced yes)
 		(effects
@@
 		)
 		(property "Intersheetrefs" "${INTERSHEET_REFS}"
-			(at 91.8645 43.18 0)
+			(at 124.8845 43.18 0)
 			(hide yes)
 			(show_name no)
@@
 	(global_label "SPI_CLK/CCLK"
 		(shape bidirectional)
-		(at 74.93 45.72 0)
+		(at 107.95 45.72 0)
 		(fields_autoplaced yes)
 		(effects
@@
 		)
 		(property "Intersheetrefs" "${INTERSHEET_REFS}"
-			(at 92.457 45.72 0)
+			(at 125.477 45.72 0)
 			(hide yes)
 			(show_name no)
@@
 		)
 	)
-	(global_label "SPI_CLK/CCLK"
-		(shape bidirectional)
-		(at 77.47 81.28 0)
-		(fields_autoplaced yes)
-		(effects
-			(font
-				(size 0.889 0.889)
-			)
-			(justify left)
-		)
-		(property "Intersheetrefs" "${INTERSHEET_REFS}"
-			(at 89.9894 81.28 0)
-			(hide yes)
-			(show_name no)
-			(do_not_autoplace no)
-			(effects
-				(font
-					(size 1.27 1.27)
-				)
-				(justify left)
-			)
-		)
-	)
 	(global_label "/NMI"
 		(shape bidirectional)
@@
 		)
 	)
-	(global_label "SPI_MOSI"
-		(shape bidirectional)
-		(at 77.47 76.2 0)
-		(fields_autoplaced yes)
-		(effects
-			(font
-				(size 0.889 0.889)
-			)
-			(justify left)
-		)
-		(property "Intersheetrefs" "${INTERSHEET_REFS}"
-			(at 86.391 76.2 0)
-			(hide yes)
-			(show_name no)
-			(do_not_autoplace no)
-			(effects
-				(font
-					(size 1.27 1.27)
-				)
-				(justify left)
-			)
-		)
-	)
 	(global_label "/IRQ"
 		(shape bidirectional)
@@
 		)
 	)
+	(global_label "{slash}SPI_FLASH"
+		(shape bidirectional)
+		(at 109.22 83.82 0)
+		(fields_autoplaced yes)
+		(effects
+			(font
+				(size 1.2446 1.2446)
+			)
+			(justify left)
+		)
+		(property "Intersheetrefs" "${INTERSHEET_REFS}"
+			(at 124.1393 83.82 0)
+			(hide yes)
+			(show_name no)
+			(do_not_autoplace no)
+			(effects
+				(font
+					(size 1.27 1.27)
+				)
+				(justify left)
+			)
+		)
+	)
 	(global_label "D7"
 		(shape bidirectional)
@@
 			(hide yes)
 			(show_name no)
-			(do_not_autoplace no)
-			(effects
-				(font
-					(size 1.27 1.27)
-				)
-				(justify left)
-			)
-		)
-	)
-	(global_label "SPI_MISO/DIN"
-		(shape bidirectional)
-		(at 77.47 78.74 0)
-		(fields_autoplaced yes)
-		(effects
-			(font
-				(size 0.889 0.889)
-			)
-			(justify left)
-		)
-		(property "Intersheetrefs" "${INTERSHEET_REFS}"
-			(at 89.5659 78.74 0)
-			(hide yes)
-			(show_name no)

Commit message: more layout work
Parts:
- removed IC7: 74LVC138, csa_ultracpu:SO16, symbol csa_ultracpu-eagle-import:74138D
Connections:
- net A0: now also U1.25 (A12); no longer U1.1 (A0)
- net A1: now also U1.26 (A13); no longer U1.2 (A1)
- net A2: now also U1.27 (A14); no longer U1.3 (A2)
- net A3: now also U1.28 (A18); no longer U1.4 (A3)
- net FA12: now also U1.1 (A0); no longer U1.25 (A12)
- net FA13: now also U1.2 (A1); no longer U1.26 (A13)
- net FA14: now also U1.3 (A2); no longer U1.27 (A14)
- net FA15: now also U1.4 (A3); no longer U1.42 (A15)
- net FA18: now also U1.42 (A15); no longer U1.28 (A18)
Other:
- note added: "Address line ordering to facilitate better PCB routing: FPGA only Ax on "upper" half of chip."
- note added: "CSA-ULTRACPU-V3.0A-20260905"
- note removed: "CSA-ULTRACPU-V2.2A-20260602"
