File: Board/CPU,RAM,ROM.kicad_sch (KiCad schematic)
At the start: 16 parts, among them IC1 74LVC125, IC6 741G04DBV, U1 IS61WV51216EDALL, X3 SG-8002CE

Commit message: more layout work
Connections:
- net /BE renamed /BE
Changed lines of the file:
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@@
 	(wire
 		(pts
-			(xy 171.45 186.69) (xy 158.75 186.69)
+			(xy 171.45 186.69) (xy 150.495 186.69)
 		)
 		(stroke
@@
 		)
 	)
+	(global_label "PHI2"
+		(shape bidirectional)
+		(at 150.495 186.69 180)
+		(fields_autoplaced yes)
+		(effects
+			(font
+				(size 1.2446 1.2446)
+			)
+			(justify right)
+		)
+		(property "Intersheetrefs" "${INTERSHEET_REFS}"
+			(at 142.1543 186.69 0)
+			(hide yes)
+			(show_name no)
+			(do_not_autoplace no)
+			(effects
+				(font
+					(size 1.27 1.27)
+				)
+				(justify right)
+			)
+		)
+	)
 	(global_label "A3"
 		(shape input)
@@
 		)
 	)
+	(global_label "QCLK"
+		(shape bidirectional)
+		(at 208.28 57.15 0)
+		(fields_autoplaced yes)
+		(effects
+			(font
+				(size 1.778 1.778)
+			)
+			(justify left)
+		)
+		(property "Intersheetrefs" "${INTERSHEET_REFS}"
+			(at 220.8728 57.15 0)
+			(hide yes)
+			(show_name no)
+			(do_not_autoplace no)
+			(effects
+				(font
+					(size 1.27 1.27)
+				)
+				(justify left)
+			)
+		)
+	)
 	(global_label "D4"
 		(shape bidirectional)
@@
 			(hide yes)
 			(show_name no)
+			(do_not_autoplace no)
+			(effects
+				(font
+					(size 1.27 1.27)
+				)
+				(justify left)
+			)
+		)
+	)
+	(global_label "{slash}BE"
+		(shape bidirectional)
+		(at 303.53 151.13 0)
+		(fields_autoplaced yes)
+		(effects
+			(font
+				(size 1.2446 1.2446)
+			)
+			(justify left)
+		)
+		(property "Intersheetrefs" "${INTERSHEET_REFS}"
+			(at 311.2188 151.13 0)
+			(hide yes)
+			(show_name no)

Commit message: more layout work
Connections:
- net GND: now also U$1.1 (P$1)
- net SPI_MISO/DIN: now also U$4.2 (SO)
Changed lines of the file:
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@@
 	)
 	(junction
-		(at 353.06 46.99)
-		(diameter 0)
-		(color 0 0 0 0)
-	)
-	(junction
 		(at 90.17 83.82)
 		(diameter 0)
@@
 	)
 	(junction
-		(at 353.06 74.93)
+		(at 92.71 43.18)
 		(diameter 0)
 		(color 0 0 0 0)
@@
 	)
 	(junction
+		(at 260.35 72.39)
+		(diameter 0)
+		(color 0 0 0 0)
+	)
+	(junction
+		(at 186.055 207.01)
+		(diameter 0)
+		(color 0 0 0 0)
+	)
+	(junction
 		(at 39.37 45.72)
 		(diameter 0)
@@
 	(wire
 		(pts
+			(xy 186.055 213.36) (xy 186.055 207.01)
+		)
+		(stroke
+			(width 0)
+			(type default)
+		)
+	)
+	(wire
+		(pts
 			(xy 224.79 184.15) (xy 242.57 184.15)
 		)
@@
 	(wire
 		(pts
+			(xy 92.71 43.18) (xy 92.71 78.74)
+		)
+		(stroke
+			(width 0.1524)
+			(type solid)
+		)
+	)
+	(wire
+		(pts
 			(xy 99.06 200.66) (xy 99.06 161.29)
 		)
@@
 	(wire
 		(pts
-			(xy 312.42 74.93) (xy 353.06 74.93)
+			(xy 312.42 74.93) (xy 363.22 74.93)
 		)
 		(stroke
@@
 	(wire
 		(pts
+			(xy 92.71 43.18) (xy 107.95 43.18)
+		)
+		(stroke
+			(width 0.1524)
+			(type solid)
+		)
+	)
+	(wire
+		(pts
 			(xy 46.99 176.53) (xy 55.88 176.53)
 		)
@@
 	(wire
 		(pts
-			(xy 72.39 43.18) (xy 107.95 43.18)
+			(xy 72.39 43.18) (xy 92.71 43.18)
 		)
 		(stroke
@@
 	(wire
 		(pts
-			(xy 181.61 207.01) (xy 189.23 207.01)
+			(xy 181.61 207.01) (xy 186.055 207.01)
 		)
 		(stroke
@@
 	(wire
 		(pts
+			(xy 186.055 207.01) (xy 189.23 207.01)
+		)
+		(stroke
+			(width 0.1524)
+			(type solid)
+		)
+	)
+	(wire
+		(pts
 			(xy 227.33 224.79) (xy 227.33 219.71)
 		)
@@
 	(wire
 		(pts
-			(xy 353.06 74.93) (xy 363.22 74.93)
-		)
-		(stroke
-			(width 0.1524)
-			(type solid)
-		)
-	)
-	(wire
-		(pts
 			(xy 184.15 161.29) (xy 171.45 161.29)
 		)
@@
 	(wire
 		(pts
+			(xy 260.35 72.39) (xy 271.78 72.39)
+		)
+		(stroke
+			(width 0.1524)
+			(type solid)
+		)
+	)
+	(wire
+		(pts
 			(xy 91.44 185.42) (xy 91.44 176.53)
 		)
@@
 	(wire
 		(pts
-			(xy 353.06 46.99) (xy 363.22 46.99)
-		)
-		(stroke
-			(width 0.1524)
-			(type solid)
-		)
-	)
-	(wire
-		(pts
 			(xy 72.39 40.64) (xy 90.17 40.64)
 		)
@@
 	(wire
 		(pts
-			(xy 256.54 72.39) (xy 271.78 72.39)
+			(xy 256.54 72.39) (xy 260.35 72.39)
 		)
 		(stroke
@@
 	(wire
 		(pts
-			(xy 92.71 43.18) (xy 92.71 78.74)
-		)
-		(stroke
-			(width 0.1524)
-			(type solid)
-		)
-	)
-	(wire
-		(pts
 			(xy 90.17 40.64) (xy 107.95 40.64)
 		)
@@
 	(wire
 		(pts
+			(xy 189.865 213.36) (xy 186.055 213.36)
+		)
+		(stroke
+			(width 0)
+			(type default)
+		)
+	)
+	(wire
+		(pts
 			(xy 214.63 130.81) (xy 222.25 130.81)
 		)
@@
 	(wire
 		(pts
-			(xy 353.06 52.07) (xy 353.06 46.99)
-		)
-		(stroke
-			(width 0.1524)
-			(type solid)
-		)
-	)
-	(wire
-		(pts
 			(xy 86.36 195.58) (xy 96.52 195.58)
 		)
@@
 	(wire
 		(pts
-			(xy 342.9 46.99) (xy 353.06 46.99)
+			(xy 342.9 46.99) (xy 363.22 46.99)
 		)
 		(stroke
@@
 	(wire
 		(pts
-			(xy 353.06 74.93) (xy 353.06 67.31)
-		)
-		(stroke
-			(width 0.1524)
-			(type solid)
-		)
-	)
-	(wire
-		(pts
 			(xy 219.71 186.69) (xy 242.57 186.69)
 		)
@@
 	(global_label "/IRQ"
 		(shape bidirectional)
-		(at 184.15 207.01 0)
+		(at 189.865 213.36 0)
 		(fields_autoplaced yes)
 		(effects
@@
 		)
 		(property "Intersheetrefs" "${INTERSHEET_REFS}"
-			(at 192.6093 207.01 0)
+			(at 198.3243 213.36 0)
 			(hide yes)
 			(show_name no)
@@
 				)
 			)
+		)
+	)
+	(symbol
+		(lib_id "csa_ultracpu-eagle-import:W65C816SPLCC")
+		(at 260.35 69.85 0)
+		(unit 3)
+		(body_style 1)
+		(exclude_from_sim no)
+		(in_bom yes)
+		(on_board yes)
+		(in_pos_files yes)
+		(dnp no)
+		(fields_autoplaced yes)
+		(property "Reference" "U$1"
+			(at 241.935 57.785 0)
+			(hide yes)
+			(show_name no)
+			(do_not_autoplace no)
+			(effects
+				(font
+					(size 1.778 1.5113)
+				)
+				(justify left bottom)
+			)
+		)
+		(property "Value" "W65C816SPLCC"
+			(at 250.19 107.95 0)
+			(hide yes)
+			(show_name no)
+			(do_not_autoplace no)
+			(effects
+				(font
+					(size 1.778 1.5113)
+				)
+				(justify left bottom)
+			)
+		)
+		(property "Footprint" "csa_ultracpu:PLCC44"
+			(at 260.35 69.85 0)
+			(hide yes)
+			(show_name no)
+			(do_not_autoplace no)
+			(effects
+				(font
+					(size 1.27 1.27)
+				)
+			)
+		)
+		(property "Datasheet" ""
+			(at 260.35 69.85 0)
+			(hide yes)
+			(show_name no)
+			(do_not_autoplace no)
+			(effects
+				(font
+					(size 1.27 1.27)
+				)
+			)
+		)
+		(property "Description" ""
+			(at 260.35 69.85 0)
+			(hide yes)
+			(show_name no)
+			(do_not_autoplace no)
+			(effects
+				(font
+					(size 1.27 1.27)
+				)
+			)
+		)
+		(pin "10"
+		)
+		(pin "11"
+		)
+		(pin "13"
+		)
+		(pin "14"
+		)
+		(pin "15"
+		)
+		(pin "16"
+		)
+		(pin "17"
+		)
+		(pin "18"
+		)
+		(pin "19"
+		)
+		(pin "2"
+		)
+		(pin "20"
+		)
+		(pin "21"
+		)
+		(pin "22"
+		)
+		(pin "23"
+		)
+		(pin "25"
+		)
+		(pin "26"
+		)
+		(pin "27"
+		)
+		(pin "28"
+		)
+		(pin "29"
+		)
+		(pin "3"
+		)
+		(pin "30"
+		)
+		(pin "31"
+		)
+		(pin "32"
+		)
+		(pin "33"
+		)
+		(pin "34"
+		)
+		(pin "35"
+		)
+		(pin "36"
+		)
+		(pin "37"
+		)
+		(pin "38"
+		)
+		(pin "39"
+		)
+		(pin "4"
+		)
+		(pin "40"
+		)
+		(pin "41"
+		)
+		(pin "42"
+		)
+		(pin "43"
+		)
+		(pin "44"
+		)
+		(pin "5"
+		)
+		(pin "6"
+		)
+		(pin "7"
+		)
+		(pin "8"
+		)
+		(pin "24"
+		)
+		(pin "9"
+		)
+		(pin "1"
+		)
+		(instances
+			(project "csa_ultracpu"
+				(path "/381336a5-a662-4c84-a650-90475fa59a97/eedf0d8e-348e-4413-8cbb-f9fc41eecd37"
+					(reference "U$1")
+					(unit 3)
+				)
+			)

Commit message: more layout work, first candidate
Parts:
- added unit 3 of U$1
Connections:
- net GND: now also U$1.1 (P$1); no longer U$1.1 (P$1)

Commit message: layout done
Parts:
- IC1: LCSC (none) -> C6057
- IC6: LCSC (none) -> C434067
- JP7: LCSC (none) -> C587039
- R10, R11, R3, R9: LCSC (none) -> C17414
- U$1: LCSC (none) -> C72279
- U$18, U$4: LCSC (none) -> C72124
- U1: LCSC (none) -> C57407
- X3: LCSC (none) -> C2831398
Changed lines of the file:
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@@
+			)
+		)
+		(property "LCSC" "C72124"
+			(at 54.61 35.56 0)
+			(hide yes)
+			(show_name no)
+			(do_not_autoplace no)
+			(effects
+				(font
+					(size 1.27 1.27)
+				)
 			)
 		)
@@
 			)
 		)
+		(property "LCSC" "C17414"
+			(at 215.6714 218.44 0)
+			(hide yes)
+			(show_name no)
+			(do_not_autoplace no)
+			(effects
+				(font
+					(size 1.27 1.27)
+				)
+			)
+		)
 		(pin "1"
 		)
@@
 			)
 		)
+		(property "LCSC" "C17414"
+			(at 225.8314 218.44 0)
+			(hide yes)
+			(show_name no)
+			(do_not_autoplace no)
+			(effects
+				(font
+					(size 1.27 1.27)
+				)
+			)
+		)
 		(pin "1"
 		)
@@
 			)
 		)
+		(property "LCSC" "C72124"
+			(at 54.61 71.12 0)
+			(hide yes)
+			(show_name no)
+			(do_not_autoplace no)
+			(effects
+				(font
+					(size 1.27 1.27)
+				)
+			)
+		)
 		(pin "1"
 		)
@@
 			)
 		)
+		(property "LCSC" "C17414"
+			(at 156.4386 48.26 0)
+			(hide yes)
+			(show_name no)
+			(do_not_autoplace no)
+			(effects
+				(font
+					(size 1.27 1.27)
+				)
+			)
+		)
 		(pin "1"
 		)
@@
 		(property "Description" ""
 			(at 199.39 153.67 0)
+			(hide yes)
+			(show_name no)
+			(do_not_autoplace no)
+			(effects
+				(font
+					(size 1.27 1.27)
+				)
+			)
+		)
+		(property "LCSC" "C72279"
+			(at 180.975 141.605 0)
 			(hide yes)
 			(show_name no)
@@
 			)
 		)
+		(property "LCSC" "C2831398"
+			(at 181.61 50.8314 0)
+			(hide yes)
+			(show_name no)
+			(do_not_autoplace no)
+			(effects
+				(font
+					(size 1.27 1.27)
+				)
+			)
+		)
 		(pin "2"
 		)
@@
 			)
 		)
+		(property "LCSC" "C57407"
+			(at 71.9933 153.67 0)
+			(hide yes)
+			(show_name no)
+			(do_not_autoplace no)
+			(effects
+				(font
+					(size 1.27 1.27)
+				)
+			)
+		)
 		(pin "34"
 		)
@@
 			)
 		)
+		(property "LCSC" "C6057"
+			(at 332.105 125.095 0)
+			(hide yes)
+			(show_name no)
+			(do_not_autoplace no)
+			(effects
+				(font
+					(size 1.27 1.27)
+				)
+			)
+		)
 		(pin "1"
 		)
@@
 		(property "Description" ""
 			(at 269.24 74.93 0)
+			(hide yes)
+			(show_name no)
+			(do_not_autoplace no)
+			(effects
+				(font
+					(size 1.27 1.27)
+				)
+			)
+		)
+		(property "LCSC" "C72279"
+			(at 250.825 62.865 0)
 			(hide yes)
 			(show_name no)
@@
 			)
 		)
+		(property "LCSC" "C72279"
+			(at 241.935 57.785 0)
+			(hide yes)
+			(show_name no)
+			(do_not_autoplace no)
+			(effects
+				(font
+					(size 1.27 1.27)
+				)
+			)
+		)
 		(pin "10"
 		)
@@
 			)
 		)
+		(property "LCSC" "C6057"
+			(at 362.585 60.325 0)
+			(hide yes)
+			(show_name no)
+			(do_not_autoplace no)
+			(effects
+				(font
+					(size 1.27 1.27)
+				)
+			)
+		)
 		(pin "1"
 		)
@@
 			)
 		)
+		(property "LCSC" "C434067"
+			(at 311.785 62.865 0)
+			(hide yes)
+			(show_name no)
+			(do_not_autoplace no)
+			(effects
+				(font
+					(size 1.27 1.27)
+				)
+			)
+		)
 		(pin "2"
 		)
@@
 			)
 		)
+		(property "LCSC" "C434067"
+			(at 271.145 150.495 0)
+			(hide yes)
+			(show_name no)
+			(do_not_autoplace no)
+			(effects
+				(font
+					(size 1.27 1.27)
+				)
+			)
+		)
 		(pin "3"
 		)
@@
 			)
 		)
+		(property "LCSC" "C587039"
+			(at 245.11 180.34 0)
+			(hide yes)
+			(show_name no)
+			(do_not_autoplace no)
+			(effects
+				(font
+					(size 1.27 1.27)
+				)
+			)
+		)
 		(pin "1"
 		)
@@
 			(hide yes)
 			(show_name no)
+			(do_not_autoplace no)
+			(effects
+				(font
+					(size 1.27 1.27)
+				)
+			)
+		)
+		(property "LCSC" "C17414"
+			(at 180.1114 218.44 0)
+			(hide yes)
+			(show_name no)

Commit message: test release
Connections:
- net ABORTB renamed /ABORT
Changed lines of the file:
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@@
+	)
+	(junction
+		(at 224.79 167.64)
+		(diameter 0)
+		(color 0 0 0 0)
 	)
 	(junction
@@
 	(wire
 		(pts
-			(xy 224.79 163.83) (xy 224.79 184.15)
+			(xy 224.79 163.83) (xy 224.79 167.64)
 		)
 		(stroke
@@
 	(wire
 		(pts
+			(xy 235.585 167.64) (xy 224.79 167.64)
+		)
+		(stroke
+			(width 0)
+			(type default)
+		)
+	)
+	(wire
+		(pts
 			(xy 214.63 135.89) (xy 222.25 135.89)
 		)
@@
 	(wire
 		(pts
+			(xy 224.79 167.64) (xy 224.79 184.15)
+		)
+		(stroke
+			(width 0.1524)
+			(type solid)
+		)
+	)
+	(wire
+		(pts
 			(xy 184.15 173.99) (xy 153.67 173.99)
 		)
@@
 			(width 0.1524)
 			(type solid)
+		)
+	)
+	(wire
+		(pts
+			(xy 224.79 167.64) (xy 224.79 167.005)
+		)
+		(stroke
+			(width 0)
+			(type default)
 		)
 	)
@@
 			)
 		)
+	)
+	(global_label "{slash}ABORT"
+		(shape bidirectional)
+		(at 235.585 167.64 0)
+		(fields_autoplaced yes)
+		(effects
+			(font
+				(size 0.889 0.889)
+			)
+			(justify left)
+		)
+		(property "Intersheetrefs" "${INTERSHEET_REFS}"
+			(at 243.5323 167.64 0)
+			(hide yes)
+			(show_name no)
+			(do_not_autoplace no)
+			(effects
+				(font
+					(size 1.27 1.27)
+				)
+				(justify left)
+			)
+		)
