File: Board/Power.kicad_sch (KiCad schematic)
At the start: 76 parts

Commit message: update
Parts:
- DS1818: footprint csa_ultracpu:TO92 -> Package_TO_SOT_SMD:SOT-23
Changed lines of the file:
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@@
 			)
 		)
-		(property "Footprint" "csa_ultracpu:TO92"
+		(property "Footprint" "Package_TO_SOT_SMD:SOT-23"
 			(at 259.08 96.52 0)
 			(effects

Commit message: more layout work
Other:
- note added: "CSA-ULTRACPU-V3.0A"
- note removed: "CSA-ULTRACPU-V2.2A"
Changed lines of the file:
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@@
 		)
 	)
-	(text "CSA-ULTRACPU-V2.2A"
+	(text "CSA-ULTRACPU-V3.0A"
 		(exclude_from_sim no)
 		(at 251.46 175.26 0)

Commit message: more layout work
Connections:
- net V12: now also C36.1
- net V33: no longer C36.1
Changed lines of the file:
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@@
-	)
-	(junction
-		(at 139.7 170.18)
-		(diameter 0)
-		(color 0 0 0 0)
 	)
 	(junction
@@
 	)
 	(junction
+		(at 154.94 160.02)
+		(diameter 0)
+		(color 0 0 0 0)
+	)
+	(junction
 		(at 99.06 154.94)
 		(diameter 0)
@@
 	(wire
 		(pts
+			(xy 154.94 160.02) (xy 158.75 160.02)
+		)
+		(stroke
+			(width 0.1524)
+			(type solid)
+		)
+	)
+	(wire
+		(pts
 			(xy 35.56 154.94) (xy 55.88 154.94)
 		)
@@
 	(wire
 		(pts
-			(xy 147.32 160.02) (xy 158.75 160.02)
+			(xy 147.32 160.02) (xy 154.94 160.02)
 		)
 		(stroke
@@
 	(wire
 		(pts
+			(xy 154.94 160.02) (xy 154.94 172.72)
+		)
+		(stroke
+			(width 0.1524)
+			(type solid)
+		)
+	)
+	(wire
+		(pts
 			(xy 297.18 45.72) (xy 302.26 45.72)
 		)
@@
 	(wire
 		(pts
-			(xy 154.94 170.18) (xy 154.94 172.72)
-		)
-		(stroke
-			(width 0.1524)
-			(type solid)
-		)
-	)
-	(wire
-		(pts
 			(xy 142.24 73.66) (xy 152.4 73.66)
 		)
@@
 		)
 		(stroke
-			(width 0.1524)
-			(type solid)
-		)
-	)
-	(wire
-		(pts
-			(xy 139.7 170.18) (xy 154.94 170.18)
-		)
-		(stroke
