File: Board/Power.kicad_sch (KiCad schematic)
At the start: 76 parts

Commit message: layout done
Parts:
- C1, C120, C123, C14, C4, C49, C54, C55, C56, C57: LCSC (none) -> C15849
- C101, C102, C103, C104, C105, C106, C107, C108, C109, C11, C110, C111, C112, C113, C12, C121, C13, C15, C17, C18, C19, C2, C20, C22, C24, C25, C26, C28, C31, C32, C34, C35, C36, C37, C41, C42, C43, C44, C45, C46, C47, C48, C58, C7, C8: LCSC (none) -> C14663
- C38, C5, C64, C65, C66, C67, C68, C69, C70, C71: LCSC (none) -> C45783
- C6: footprint csa_ultracpu:E2,5-6 -> Capacitor_SMD:C_0805_2012Metric_Pad1.18x1.45mm_HandSolder; LCSC (none) -> C16780
- DS1818: LCSC (none) -> C143298
- LED1: LCSC (none) -> C85161
- R22: footprint csa_ultracpu:0207_2V -> Resistor_SMD:R_0603_1608Metric_Pad0.98x0.95mm_HandSolder; LCSC (none) -> C23151
- R24: LCSC (none) -> C17414
- S1: LCSC (none) -> C231320
- U$16: LCSC (none) -> C338874
- U$3: LCSC (none) -> C6186
Connections:
- net GND: now also C6.2 (-); no longer C6.-
- net VCC: now also C6.1 (+); no longer C6.+
