File: Board/fpga_io.kicad_sch (KiCad schematic)
At the start: 2 parts, among them IC1 74LVC125, U2 XC6SLX25T-CSG324

Commit message: layout work
Connections:
- net /RAMWE: now also U2.P8 (IO_L44N_2)
- net HDMI-CK+: now also U2.V4 (IO_L63N_2)
- net HDMI-CK-: now also U2.T4 (IO_L63P_2)
- net HDMI-D0+: now also U2.V5 (IO_L49N_D4_2)
- net HDMI-D0-: now also U2.U5 (IO_L49P_D3_2)
- net HDMI-D1+: now also U2.V7 (IO_L43N_2)
- net HDMI-D1-: now also U2.U7 (IO_L43P_2)
- net HDMI-D2+: now also U2.V8 (IO_L41N_VREF_2)
- net HDMI-D2-: now also U2.U8 (IO_L41P_2)
- net RAMA5: now also U2.U10 (IO_L30P_GCLK1_D13_2)
- net RAMA6: now also U2.R8 (IO_L31P_GCLK31_D14_2)
- net RAMA7: now also U2.V9 (IO_L32N_GCLK28_2)
- net RAMA8: now also U2.T8 (IO_L31N_GCLK30_D15_2)
- net RAMA9: now also U2.V6 (IO_L45N_2)
- net V33: now also U2.E2 (VCCO_3), U2.G4 (VCCO_3), U2.J2 (VCCO_3), U2.J5 (VCCO_3), U2.M4 (VCCO_3), U2.P9 (VCCO_2), U2.R12 (VCCO_2), U2.R2 (VCCO_3), U2.R6 (VCCO_2), U2.U14 (VCCO_2), U2.U4 (VCCO_2), U2.U9 (VCCO_2)

Commit message: layout work
Connections:
- net /RAMCS: now also U2.P11 (IO_L20N_2)
- net GND: now also IC1.5 (I)
- net RAMA0: now also U2.V14 (IO_L12N_D2_MISO3_2)
- net RAMA1: now also U2.V15 (IO_L5N_2)
- net RAMA10: now also U2.T14 (IO_L12P_D1_MISO2_2)
- net RAMA11: now also U2.N14 (IO_L53N_VREF_1)
- net RAMA12: now also U2.U15 (IO_L5P_2)
- net RAMA13: now also U2.T15 (IO_L1N_M0_CMPMISO_2)
- net RAMA14: now also U2.V16 (IO_L2N_CMPMOSI_2)
- net RAMA15: now also U2.N18 (IO_L48N_M1DQ9_1)
- net RAMA16: now also U2.N17 (IO_L48P_HDC_M1DQ8_1)
- net RAMA17: now also U2.M18 (IO_L47N_LDC_M1DQ1_1)
- net RAMA18: now also U2.U16 (IO_L2P_CMPCLK_2)
- net RAMA2: now also U2.U13 (IO_L14P_D11_2)
- net RAMA3: now also U2.V13 (IO_L14N_D12_2)
- net RAMA4: now also U2.P12 (IO_L13N_D10_2)
- net RAMD0: now also U2.T12 (IO_L19P_2)
- net RAMD1: now also U2.R11 (IO_L16P_2)
- net RAMD2: now also U2.V12 (IO_L19N_2)
- net RAMD3: now also U2.V11 (IO_L23N_2)
- net RAMD4: now also U2.R10 (IO_L29P_GCLK3_2)
- net RAMD5: now also U2.T11 (IO_L16N_VREF_2)
- net RAMD6: now also U2.T10 (IO_L29N_GCLK2_2)
- net RAMD7: now also U2.V10 (IO_L30N_GCLK0_USERCCLK_2)
- net SPI_CLK/CCLK: now also U2.R15 (IO_L1P_CCLK_2)
- net SPI_MISO/DIN: now also U2.R13 (IO_L3P_D0_DIN_MISO_MISO1_2)
- net SPI_MOSI: now also U2.T13 (IO_L3N_MOSI_CSI_B_MISO0_2)
- net at U2.N12 (IO_L13P_M1_2): now also IC1.6 (O)
- net /FPGA_BOOT: now reaches U2.V3 (IO_L65N_CSO_B_2)
- net RAMD15: now reaches U2.N15 (IO_L50P_M1UDQS_1)
- net /RAMLB: now reaches U2.N16 (IO_L50N_M1UDQSN_1)
- net RAMD12: now reaches U2.P15 (IO_L74P_AWAKE_1)
- net RAMD13: now reaches U2.P16 (IO_L74N_DOUT_BUSY_1)
- net /RAMUB: now reaches U2.P17 (IO_L49P_M1DQ10_1)
- net RAMD14: now reaches U2.P18 (IO_L49N_M1DQ11_1)
- net RAMD10: now reaches U2.T17 (IO_L51P_M1DQ12_1)
- net RAMD11: now reaches U2.T18 (IO_L51N_M1DQ13_1)
- net RAMD8: now reaches U2.U17 (IO_L52P_M1DQ14_1)
- net RAMD9: now reaches U2.U18 (IO_L52N_M1DQ15_1)
Other:
- moved on the sheet: IC1A, IC1B, U2A

Commit message: replace Spartan6 xc6slx25t with cheaper xc6slx65, start re-layout
Parts:
- removed U2: XC6SLX25T-CSG324, Package_BGA:Xilinx_CSGA324, symbol FPGA_Xilinx_Spartan6:XC6SLX25T-CSG324
- added U4: XC6SLX25-CSG324, Package_BGA:Xilinx_CSG324, symbol FPGA_Xilinx_Spartan6:XC6SLX25-CSG324
Connections:
- net HDMI-CK+: now also U4.V4 (IO_L63N_2)
- net HDMI-CK-: now also U4.T4 (IO_L63P_2)
- net HDMI-D0+: now also U4.V5 (IO_L49N_D4_2)
- net HDMI-D0-: now also U4.U5 (IO_L49P_D3_2)
- net HDMI-D1+: now also U4.V7 (IO_L43N_2)
- net HDMI-D1-: now also U4.U7 (IO_L43P_2)
- net HDMI-D2+: now also U4.V8 (IO_L41N_VREF_2)
- net HDMI-D2-: now also U4.U8 (IO_L41P_2)
- net RAMA5: now also U4.U10 (IO_L30P_GCLK1_D13_2)
- net RAMA9: now also U4.V6 (IO_L45N_2)
- net V33: now also U4.B10 (VCCO_0), U4.B15 (VCCO_0), U4.B5 (VCCO_0), U4.D13 (VCCO_0), U4.D7 (VCCO_0), U4.E10 (VCCO_0), U4.E17 (VCCO_1), U4.E2 (VCCO_3), U4.G15 (VCCO_1), U4.G4 (VCCO_3), U4.J14 (VCCO_1), U4.J17 (VCCO_1), U4.J2 (VCCO_3), U4.J5 (VCCO_3), U4.M15 (VCCO_1), U4.M4 (VCCO_3), U4.P9 (VCCO_2), U4.R12 (VCCO_2), U4.R17 (VCCO_1), U4.R2 (VCCO_3), U4.R6 (VCCO_2), U4.U14 (VCCO_2), U4.U4 (VCCO_2), U4.U9 (VCCO_2)
- net at IC1.3 (O): now also U4.D4 (IO_L1P_HSWAPEN_0)

Commit message: more layout work
Connections:
- net A0: now also U4.F11 (IO_L42P_0)
- net A1: now also U4.E11 (IO_L42N_0)
- net A2: now also U4.F10 (IO_L40N_0)
- net A3: now also U4.C10 (IO_L37P_GCLK13_0)
- net A4: now also U4.C9 (IO_L34N_GCLK18_0)
Changed lines of the file:
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@@
 	(wire
 		(pts
-			(xy 454.66 137.16) (xy 454.66 182.88)
-		)
-		(stroke
-			(width 0.1524)
-			(type solid)
-		)
-	)
-	(wire
-		(pts
 			(xy 441.96 137.16) (xy 441.96 147.32)
 		)
@@
 	(wire
 		(pts
+			(xy 8.255 99.06) (xy 15.24 99.06)
+		)
+		(stroke
+			(width 0)
+			(type default)
+		)
+	)
+	(wire
+		(pts
 			(xy 396.24 137.16) (xy 396.24 167.64)
 		)
@@
 	(wire
 		(pts
+			(xy 8.89 137.16) (xy 15.24 137.16)
+		)
+		(stroke
+			(width 0)
+			(type default)
+		)
+	)
+	(wire
+		(pts
 			(xy 426.72 58.42) (xy 426.72 35.56)
 		)
@@
 	(wire
 		(pts
-			(xy 459.74 182.88) (xy 459.74 137.16)
-		)
-		(stroke
-			(width 0.1524)
-			(type solid)
-		)
-	)
-	(wire
-		(pts
 			(xy 190.5 13.97) (xy 190.5 21.59)
 		)
@@
 	(wire
 		(pts
+			(xy 8.255 111.76) (xy 15.24 111.76)
+		)
+		(stroke
+			(width 0)
+			(type default)
+		)
+	)
+	(wire
+		(pts
 			(xy 355.6 142.24) (xy 350.52 142.24)
 		)
@@
 	(wire
 		(pts
+			(xy 8.89 139.7) (xy 15.24 139.7)
+		)
+		(stroke
+			(width 0)
+			(type default)
+		)
+	)
+	(wire
+		(pts
 			(xy 401.32 144.78) (xy 403.86 144.78)
 		)
@@
 	(wire
 		(pts
-			(xy 457.2 182.88) (xy 457.2 137.16)
-		)
-		(stroke
-			(width 0.1524)
-			(type solid)
-		)
-	)
-	(wire
-		(pts
 			(xy 381 53.34) (xy 381 35.56)
 		)
@@
 	(wire
 		(pts
+			(xy 8.255 129.54) (xy 15.24 129.54)
+		)
+		(stroke
+			(width 0)
+			(type default)
+		)
+	)
+	(wire
+		(pts
 			(xy 403.86 147.32) (xy 403.86 167.64)
 		)
@@
 	(global_label "A2"
 		(shape bidirectional)
-		(at 459.74 177.8 90)
+		(at 8.255 129.54 180)
 		(fields_autoplaced yes)
 		(effects
@@
 				(size 1.2446 1.2446)
 			)
-			(justify left)
+			(justify right)
 		)
 		(property "Intersheetrefs" "${INTERSHEET_REFS}"
-			(at 459.74 171.5337 90)
+			(at 1.9887 129.54 0)
 			(hide yes)
 			(show_name no)
@@
 					(size 1.27 1.27)
 				)
-				(justify left)
+				(justify right)
 			)
 		)
@@
 	(global_label "A1"
 		(shape bidirectional)
-		(at 462.28 171.45 270)
+		(at 8.89 139.7 180)
 		(fields_autoplaced yes)
 		(effects
@@
 		)
 		(property "Intersheetrefs" "${INTERSHEET_REFS}"
-			(at 462.28 177.7163 90)
+			(at 2.6237 139.7 0)
 			(hide yes)
 			(show_name no)
@@
 	(global_label "A0"
 		(shape bidirectional)
-		(at 386.08 177.8 90)
+		(at 8.89 137.16 180)
 		(fields_autoplaced yes)
 		(effects
@@
 				(size 1.2446 1.2446)
 			)
-			(justify left)
+			(justify right)
 		)
 		(property "Intersheetrefs" "${INTERSHEET_REFS}"
-			(at 386.08 171.5337 90)
+			(at 2.6237 137.16 0)
 			(hide yes)
 			(show_name no)
@@
 					(size 1.27 1.27)
 				)
-				(justify left)
+				(justify right)
 			)
 		)
@@
 	(global_label "A4"
 		(shape bidirectional)
-		(at 457.2 177.8 90)
+		(at 8.255 99.06 180)
 		(fields_autoplaced yes)
 		(effects
@@
 				(size 1.2446 1.2446)
 			)
-			(justify left)
+			(justify right)
 		)
 		(property "Intersheetrefs" "${INTERSHEET_REFS}"
-			(at 457.2 171.5337 90)
+			(at 1.9887 99.06 0)
 			(hide yes)
 			(show_name no)
@@
 					(size 1.27 1.27)
 				)
-				(justify left)
+				(justify right)
 			)
 		)
@@
 	(global_label "A3"
 		(shape bidirectional)
-		(at 454.66 177.8 90)
+		(at 8.255 111.76 180)
 		(fields_autoplaced yes)
 		(effects
@@
 				(size 1.2446 1.2446)
 			)
-			(justify left)
+			(justify right)
 		)
 		(property "Intersheetrefs" "${INTERSHEET_REFS}"
-			(at 454.66 171.5337 90)
+			(at 1.9887 111.76 0)
 			(hide yes)
 			(show_name no)
@@
 					(size 1.27 1.27)
 				)
-				(justify left)
+				(justify right)
 			)
 		)

Commit message: more layout work
Connections:
- net /RES: now also U4.A15 (IO_L64N_SCP4_0)
- net A0: now also U4.M1 (IO_L36N_M3DQ9_3); no longer U4.F11 (IO_L42P_0)
- net A1: now also U4.T1 (IO_L33N_M3DQ13_3); no longer U4.E11 (IO_L42N_0)
- net A10: now also U4.K2 (IO_L38P_M3DQ2_3)
- net A11: now also U4.K1 (IO_L38N_M3DQ3_3)
- net A12: now also U4.J1 (IO_L40N_M3DQ7_3)
- net A13: now also U4.H2 (IO_L41P_GCLK27_M3DQ4_3)
- net A14: now also U4.H1 (IO_L41N_GCLK26_M3DQ5_3)
- net A15: now also U4.F1 (IO_L48N_M3BA1_3)
- net A2: now also U4.P2 (IO_L34P_M3UDQS_3); no longer U4.F10 (IO_L40N_0)
- net A3: now also U4.N2 (IO_L35P_M3DQ10_3); no longer U4.C10 (IO_L37P_GCLK13_0)
- net A4: now also U4.P1 (IO_L34N_M3UDQSN_3); no longer U4.C9 (IO_L34N_GCLK18_0)
- net A5: now also U4.N1 (IO_L35N_M3DQ11_3)
- net A6: now also U4.N3 (IO_L1N_VREF_3)
- net A7: now also U4.L2 (IO_L37P_M3DQ0_3)
- net A9: now also U4.L1 (IO_L37N_M3DQ1_3)
- net FA15: now also U4.C10 (IO_L37P_GCLK13_0)
- net FA16: now also U4.A11 (IO_L39N_0)
- net FA17: now also U4.C11 (IO_L36N_GCLK14_0)
- net FA18: now also U4.C9 (IO_L34N_GCLK18_0)
- net SPI_ACLK: now also U4.T2 (IO_L33P_M3DQ12_3)
- net SPI_AMOSI: now also U4.U2 (IO_L32P_M3DQ14_3)
- net SPI_NAUDIO: now also U4.U1 (IO_L32N_M3DQ15_3)
- net VPA: now also U4.P4 (IO_L2P_3)
- net /FRAMUB: now reaches U4.A10 (IO_L37N_GCLK12_0)
- net /FRAMSEL: now reaches U4.B11 (IO_L39P_0)
- net /FRAMLB: now reaches U4.B9 (IO_L35P_GCLK17_0)
- new net FA12: U4.F11 (IO_L42P_0)
- new net FA13: U4.E11 (IO_L42N_0)
- new net FA14: U4.F10 (IO_L40N_0)

Commit message: more layout work
Connections:
- net /BE_DOUT: now also U4.B8 (IO_L33P_0)
- net /BE_OUT: now also U4.B9 (IO_L35P_GCLK17_0)
- net /IOSEL: now also U4.A9 (IO_L35N_GCLK16_0)
- net /IRQ: now also U4.E16 (IO_L33P_A15_M1A10_1)
- net /LDAC: now also U4.T3 (IO_L62N_D6_2)
- net /MEMSEL: now also U4.A16 (IO_L66N_SCP0_0)
- net /RAMCS: now also U4.P11 (IO_L20N_2)
- net /RAMWE: now also U4.P8 (IO_L44N_2)
- net A8: now also U4.R5 (IO_L48P_D7_2)
- net BE_IN: now also U4.A13 (IO_L50N_0)
- net C2PHI2: now also U4.C17 (IO_L29P_A23_M1A13_1)
- net C8PHI2: now also U4.C18 (IO_L29N_A22_M1A14_1)
- net CPHI2: now also U4.D18 (IO_L31N_A18_M1A12_1)
- net D0: now also U4.A5 (IO_L6N_0)
- net D1: now also U4.C5 (IO_L6P_0)
- net D2: now also U4.A4 (IO_L5N_0)
- net D3: now also U4.B4 (IO_L5P_0)
- net D4: now also U4.A3 (IO_L4N_0)
- net D5: now also U4.B3 (IO_L4P_0)
- net D6: now also U4.A2 (IO_L2N_0)
- net D7: now also U4.B2 (IO_L2P_0)
- net E: now also U4.E1 (IO_L50N_M3BA2_3)
- net EXTIO: now also U4.A14 (IO_L62N_VREF_0)
- net FA16: now also U4.C8 (IO_L11N_0); no longer U4.A11 (IO_L39N_0)
- net FA17: now also U4.A8 (IO_L33N_0); no longer U4.C11 (IO_L36N_GCLK14_0)
- net FA19: now also U4.D2 (IO_L52P_M3A8_3)
- net GRAPHIC: now also U4.A11 (IO_L39N_0)
- net IOINH: now also U4.B14 (IO_L62P_0)
- net PET_VSYNC: now also U4.L4 (IO_L39P_M3LDQS_3)
- net PHI2: now also U4.D1 (IO_L52N_M3A9_3)
- net QCLK: now also U4.C11 (IO_L36N_GCLK14_0)
- net R/-W: now also U4.A10 (IO_L37N_GCLK12_0)
- net RAMA0: now also U4.V14 (IO_L12N_D2_MISO3_2)
- net RAMA1: now also U4.V15 (IO_L5N_2)
- net RAMA10: now also U4.T14 (IO_L12P_D1_MISO2_2)
- net RAMA11: now also U4.N14 (IO_L53N_VREF_1)
- net RAMA12: now also U4.U15 (IO_L5P_2)
- net RAMA13: now also U4.T15 (IO_L1N_M0_CMPMISO_2)
- net RAMA14: now also U4.V16 (IO_L2N_CMPMOSI_2)
- net RAMA15: now also U4.N18 (IO_L48N_M1DQ9_1)
- net RAMA16: now also U4.N17 (IO_L48P_HDC_M1DQ8_1)
- net RAMA17: now also U4.M18 (IO_L47N_LDC_M1DQ1_1)
- net RAMA18: now also U4.U16 (IO_L2P_CMPCLK_2)
- net RAMA2: now also U4.U13 (IO_L14P_D11_2)
- net RAMA3: now also U4.V13 (IO_L14N_D12_2)
- net RAMA4: now also U4.P12 (IO_L13N_D10_2)
- net RAMA6: now also U4.R8 (IO_L31P_GCLK31_D14_2)
- net RAMA7: now also U4.V9 (IO_L32N_GCLK28_2)
- net RAMA8: now also U4.T8 (IO_L31N_GCLK30_D15_2)
- net RAMD0: now also U4.T12 (IO_L19P_2)
- net RAMD1: now also U4.R11 (IO_L16P_2)
- net RAMD10: now also U4.T17 (IO_L51P_M1DQ12_1)
- net RAMD11: now also U4.T18 (IO_L51N_M1DQ13_1)
- net RAMD12: now also U4.P15 (IO_L74P_AWAKE_1)
- net RAMD13: now also U4.P16 (IO_L74N_DOUT_BUSY_1)
- net RAMD14: now also U4.P18 (IO_L49N_M1DQ11_1)
- net RAMD15: now also U4.N15 (IO_L50P_M1UDQS_1)
- net RAMD2: now also U4.V12 (IO_L19N_2)
- net RAMD3: now also U4.V11 (IO_L23N_2)
- net RAMD4: now also U4.R10 (IO_L29P_GCLK3_2)
- net RAMD5: now also U4.T11 (IO_L16N_VREF_2)
- net RAMD6: now also U4.T10 (IO_L29N_GCLK2_2)
- net RAMD7: now also U4.V10 (IO_L30N_GCLK0_USERCCLK_2)
- net RAMD8: now also U4.U17 (IO_L52P_M1DQ14_1)
- net RAMD9: now also U4.U18 (IO_L52N_M1DQ15_1)
- net RDY: now also U4.B11 (IO_L39P_0)
- net SPI_CLK/CCLK: now also U4.R15 (IO_L1P_CCLK_2)
- net SPI_IN3: now also U4.E18 (IO_L33N_A14_M1A4_1)
- net SPI_MISO/DIN: now also U4.R13 (IO_L3P_D0_DIN_MISO_MISO1_2)
- net SPI_MOSI: now also U4.T13 (IO_L3N_MOSI_CSI_B_MISO0_2)
- net SPI_NSEL2: now also U4.J18 (IO_L44N_A2_M1DQ7_1)
- net SPI_NSEL3: now also U4.K17 (IO_L45P_A1_M1LDQS_1)
- net SPI_NSEL4: now also U4.K18 (IO_L45N_A0_M1LDQSN_1)
- net SPI_NSEL5: now also U4.H17 (IO_L43P_GCLK5_M1DQ4_1)
- net SYNC: now also U4.D17 (IO_L31P_A19_M1CKE_1)
- net VDA: now also U4.E3 (IO_L50P_M3WE_3)
- net VPB: now also U4.F3 (IO_L51N_M3A4_3)
- net /FPGA_BOOT: now also U4.V3 (IO_L65N_CSO_B_2)
- net /FRAMLB: now also U4.B6 (IO_L8P_0); no longer U4.B9 (IO_L35P_GCLK17_0)
- net /FRAMSEL: now also U4.A7 (IO_L10N_0); no longer U4.B11 (IO_L39P_0)
- net /FRAMUB: now also U4.A6 (IO_L8N_VREF_0); no longer U4.A10 (IO_L37N_GCLK12_0)
- net /RAMLB: now also U4.N16 (IO_L50N_M1UDQSN_1)
- net /RAMUB: now also U4.P17 (IO_L49P_M1DQ10_1)
- net /SPI_FLASH: now also U4.H18 (IO_L43N_GCLK4_M1DQ5_1)
- net /BE: now reaches U4.F5 (IO_L55N_M3A14_3)
- net at U4.N12 (IO_L13P_M1_2): now also IC1.6 (O)

Commit message: more layout work
Connections:
- net RAMA9: now also U4.T9 (IO_L32P_GCLK29_2); no longer U4.V6 (IO_L45N_2)
- net HPD_SRC: now reaches U4.K3 (IO_L42N_GCLK24_M3LDM_3)
- net I2C_SCL: now reaches U4.L3 (IO_L39N_M3LDQSN_3)
- net I2C_SDA: now reaches U4.N4 (IO_L1P_3)
Other:
- note added: "(C) A. Fachat"
- note added: "CSA-ULTRACPU-V2.0A-20260906"
- note added: "CSA-ULTRACPU-V3.0A"
- moved on the sheet: IC1A, IC1B, U4A, U4B

Commit message: more layout work, first candidate
Connections:
- net /RAMWE: now also U4.T9 (IO_L32P_GCLK29_2); no longer U4.P8 (IO_L44N_2)
- net RAMA9: now also U4.P8 (IO_L44N_2); no longer U4.T9 (IO_L32P_GCLK29_2)
Changed lines of the file:
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@@
 	(wire
 		(pts
-			(xy 236.855 190.5) (xy 244.475 190.5)
-		)
-		(stroke
-			(width 0)
-			(type default)
-		)
-	)
-	(wire
-		(pts
 			(xy 172.72 201.93) (xy 181.61 201.93)
 		)
@@
 	(wire
 		(pts
+			(xy 236.855 190.5) (xy 244.475 190.5)
+		)
+		(stroke
+			(width 0)
+			(type default)
+		)
+	)
+	(wire
+		(pts
 			(xy 236.855 162.56) (xy 244.475 162.56)
 		)
@@
 	(wire
 		(pts
-			(xy 236.855 167.64) (xy 244.475 167.64)
-		)
-		(stroke
-			(width 0)
-			(type default)
-		)
-	)
-	(wire
-		(pts
 			(xy 236.855 119.38) (xy 244.475 119.38)
 		)
@@
 	(wire
 		(pts
+			(xy 236.855 167.64) (xy 244.475 167.64)
+		)
+		(stroke
+			(width 0)
+			(type default)
+		)
+	)
+	(wire
+		(pts
 			(xy 236.855 93.98) (xy 244.475 93.98)
 		)
@@
 	(global_label "/RAMWE"
 		(shape bidirectional)
-		(at 236.855 190.5 180)
+		(at 236.855 167.64 180)
 		(fields_autoplaced yes)
 		(effects
@@
 		)
 		(property "Intersheetrefs" "${INTERSHEET_REFS}"
-			(at 225.2546 190.5 0)
+			(at 225.2546 167.64 0)
 			(hide yes)
 			(show_name no)
@@
 	(global_label "RAMA9"
 		(shape bidirectional)
-		(at 236.855 167.64 180)
+		(at 236.855 190.5 180)
 		(fields_autoplaced yes)
 		(effects
@@
 		)
 		(property "Intersheetrefs" "${INTERSHEET_REFS}"
-			(at 226.8549 167.64 0)
+			(at 226.8549 190.5 0)
 			(hide yes)
 			(show_name no)
