File: Board/fpga_io.kicad_sch (KiCad schematic)
At the start: 2 parts, among them IC1 74LVC125, U4 XC6SLX25-CSG324

Commit message: layout done
Parts:
- IC1: LCSC (none) -> C6057
- U4: LCSC (none) -> C169795
Changed lines of the file:
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@@
+			)
+		)
+		(property "LCSC" "C169795"
+			(at 295.275 241.3 0)
+			(hide yes)
+			(show_name no)
+			(do_not_autoplace no)
+			(effects
+				(font
+					(size 1.27 1.27)
+				)
 			)
 		)
@@
 			)
 		)
+		(property "LCSC" "C6057"
+			(at 45.085 79.375 0)
+			(hide yes)
+			(show_name no)
+			(do_not_autoplace no)
+			(effects
+				(font
+					(size 1.27 1.27)
+				)
+			)
+		)
 		(pin "1"
 		)
@@
 		(property "Description" ""
 			(at 217.805 58.42 0)
+			(hide yes)
+			(show_name no)
+			(do_not_autoplace no)
+			(effects
+				(font
+					(size 1.27 1.27)
+				)
+			)
+		)
+		(property "LCSC" "C6057"
+			(at 218.44 57.785 0)
 			(hide yes)
 			(show_name no)
@@
 			(hide yes)
 			(show_name no)
+			(do_not_autoplace no)
+			(effects
+				(font
+					(size 1.27 1.27)
+				)
+			)
+		)
+		(property "LCSC" "C169795"
+			(at 121.92 234.95 0)
+			(hide yes)
+			(show_name no)

Commit message: test release
Connections:
- net /ABORT: now reaches U4.C2 (IO_L83P_3)
- net /NMI: now reaches U4.F16 (IO_L1N_A24_VREF_1)
Changed lines of the file:
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@@
+	(wire
+		(pts
+			(xy 172.72 92.71) (xy 179.07 92.71)
+		)
+		(stroke
+			(width 0)
+			(type default)
+		)
+	)
 	(wire
 		(pts
@@
 	(wire
 		(pts
+			(xy 346.075 223.52) (xy 353.695 223.52)
+		)
+		(stroke
+			(width 0)
+			(type default)
+		)
+	)
+	(wire
+		(pts
 			(xy 64.135 113.03) (xy 71.12 113.03)
 		)
@@
 		(property "Intersheetrefs" "${INTERSHEET_REFS}"
 			(at 189.8406 97.79 0)
+			(hide yes)
+			(show_name no)
+			(do_not_autoplace no)
+			(effects
+				(font
+					(size 1.27 1.27)
+				)
+				(justify left)
+			)
+		)
+	)
+	(global_label "{slash}NMI"
+		(shape bidirectional)
+		(at 179.07 92.71 0)
+		(fields_autoplaced yes)
+		(effects
+			(font
+				(size 1.2446 1.2446)
+			)
+			(justify left)
+		)
+		(property "Intersheetrefs" "${INTERSHEET_REFS}"
+			(at 187.7071 92.71 0)
 			(hide yes)
 			(show_name no)
@@
 			(hide yes)
 			(show_name no)
+			(do_not_autoplace no)
+			(effects
+				(font
+					(size 1.27 1.27)
+				)
+				(justify left)
+			)
+		)
+	)
+	(global_label "{slash}ABORT"
+		(shape bidirectional)
+		(at 353.695 223.52 0)
+		(fields_autoplaced yes)
+		(effects
+			(font
+				(size 1.2446 1.2446)
+			)
+			(justify left)
+		)
+		(property "Intersheetrefs" "${INTERSHEET_REFS}"
+			(at 364.8213 223.52 0)
+			(hide yes)
+			(show_name no)
