File: Board/fpga_support.kicad_sch (KiCad schematic)
At the start: 5 parts, among them U2 XC6SLX25T-CSG324

Commit message: replace Spartan6 xc6slx25t with cheaper xc6slx65, start re-layout
Parts:
- removed U2: XC6SLX25T-CSG324, Package_BGA:Xilinx_CSGA324, symbol FPGA_Xilinx_Spartan6:XC6SLX25T-CSG324
- added U4: XC6SLX25-CSG324, Package_BGA:Xilinx_CSG324, symbol FPGA_Xilinx_Spartan6:XC6SLX25-CSG324
Connections:
- net DONE: now also U4.V17 (DONE_2)
- net GND: now also U4.A1 (GND), U4.A18 (GND), U4.B13 (GND), U4.B7 (GND), U4.C16 (GND), U4.C3 (GND), U4.D10 (GND), U4.D5 (GND), U4.E15 (GND), U4.G12 (GND), U4.G17 (GND), U4.G2 (GND), U4.G5 (GND), U4.H10 (GND), U4.H8 (GND), U4.J11 (GND), U4.J15 (GND), U4.J4 (GND), U4.J9 (GND), U4.K10 (GND), U4.K8 (GND), U4.L11 (GND), U4.L9 (GND), U4.M17 (GND), U4.M2 (GND), U4.M6 (GND), U4.N13 (GND), U4.R1 (GND), U4.R14 (GND), U4.R18 (GND), U4.R4 (GND), U4.R9 (GND), U4.T16 (GND), U4.U12 (GND), U4.U6 (GND), U4.V1 (GND), U4.V18 (GND)
- net V12: now also U4.G7 (VCCINT), U4.H11 (VCCINT), U4.H9 (VCCINT), U4.J10 (VCCINT), U4.J8 (VCCINT), U4.K11 (VCCINT), U4.K9 (VCCINT), U4.L10 (VCCINT), U4.L8 (VCCINT), U4.M12 (VCCINT), U4.M7 (VCCINT)
- net V33: now also U4.B1 (VCCAUX), U4.B17 (VCCAUX), U4.E14 (VCCAUX), U4.E5 (VCCAUX), U4.E9 (VCCAUX), U4.G10 (VCCAUX), U4.J12 (VCCAUX), U4.K7 (VCCAUX), U4.M9 (VCCAUX), U4.P10 (VCCAUX), U4.P14 (VCCAUX), U4.P5 (VCCAUX)
- net at U$2.1 (TCK): now also U4.A17 (TCK)
- net at U$2.3 (TDO): now also U4.D16 (TDO)
- net at U$2.5 (TMS): now also U4.B18 (TMS)
- net at U$2.9 (TDI): now also U4.D15 (TDI)
- net at JP3.2, R18.1: now also U4.V2 (PROGRAM_B_2)
Other:
- note removed: "Dedicated Differential Clock input - no I/O See UG393"
- note removed: "Multi Gigabit Transceiver Pins See UG386"

Commit message: more layout work
Other:
- note added: "CSA-ULTRACPU-V2.0A-20260905"
- note added: "CSA-ULTRACPU-V3.0A"
- note removed: "CSA-ULTRACPU-V2.1A-20241207"
- note removed: "CSA-ULTRACPU-V2.2A"
Changed lines of the file:
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@@
 		)
 	)
-	(text "CSA-ULTRACPU-V2.2A"
+	(text "CSA-ULTRACPU-V3.0A"
 		(exclude_from_sim no)
 		(at 15.24 171.45 0)
@@
 		)
 	)
-	(text "CSA-ULTRACPU-V2.1A-20241207"
+	(text "CSA-ULTRACPU-V2.0A-20260905"
 		(exclude_from_sim no)
 		(at 15.24 194.31 0)

Commit message: more layout work
Parts:
- R15: footprint csa_ultracpu:0207_2V -> Capacitor_SMD:C_0603_1608Metric_Pad1.08x0.95mm_HandSolder; LCSC (none) -> C23138
Changed lines of the file:
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@@
 			)
 		)
-		(property "Footprint" "csa_ultracpu:0207_2V"
+		(property "Footprint" "Capacitor_SMD:C_0603_1608Metric_Pad1.08x0.95mm_HandSolder"
 			(at 154.94 124.46 0)
 			(hide yes)
@@
 			(at 154.94 124.46 0)
 			(hide yes)
+			(show_name no)
+			(do_not_autoplace no)
+			(effects
+				(font
+					(size 1.27 1.27)
+				)
+			)
+		)
+		(property "LCSC" "C23138"
+			(at 154.94 124.46 0)
+			(hide yes)

Commit message: more layout work
Connections:
- net GND: now also U$2.10
Other:
- note added: "CSA-ULTRACPU-V2.0A-20260906"
- note removed: "CSA-ULTRACPU-V2.0A-20260905"
- moved on the sheet: JP3, R15, R18, U4C

Commit message: more layout work, first candidate
Parts:
- added unit 1 of U$2
Connections:
- net at U4.A17 (TCK): now also U$2.1 (TCK); no longer U$2.1 (TCK)
- net at U4.D16 (TDO): now also U$2.3 (TDO); no longer U$2.3 (TDO)
- net at U4.B18 (TMS): now also U$2.5 (TMS); no longer U$2.5 (TMS)
- net at U4.D15 (TDI): now also U$2.9 (TDI); no longer U$2.9 (TDI)

Commit message: layout done
Parts:
- JP3: LCSC (none) -> C234182
- R18: LCSC (none) -> C17414
- U$2: LCSC (none) -> C5661
- U4: LCSC (none) -> C169795
Changed lines of the file:
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@@
+			)
+		)
+		(property "LCSC" "C5661"
+			(at 219.075 99.06 0)
+			(hide yes)
+			(show_name no)
+			(do_not_autoplace no)
+			(effects
+				(font
+					(size 1.27 1.27)
+				)
 			)
 		)
@@
 		(property "Description" ""
 			(at 210.82 107.95 0)
+			(hide yes)
+			(show_name no)
+			(do_not_autoplace no)
+			(effects
+				(font
+					(size 1.27 1.27)
+				)
+			)
+		)
+		(property "LCSC" "C5661"
+			(at 192.405 95.885 0)
 			(hide yes)
 			(show_name no)
@@
 			)
 		)
+		(property "LCSC" "C169795"
+			(at 269.5575 69.8499 0)
+			(hide yes)
+			(show_name no)
+			(do_not_autoplace no)
+			(effects
+				(font
+					(size 1.27 1.27)
+				)
+			)
+		)
 		(pin "A2"
 		)
@@
 			)
 		)
+		(property "LCSC" "C169795"
+			(at 60.96 62.23 0)
+			(hide yes)
+			(show_name no)
+			(do_not_autoplace no)
+			(effects
+				(font
+					(size 1.27 1.27)
+				)
+			)
+		)
 		(pin "A2"
 		)
@@
 			)
 		)
+		(property "LCSC" "C234182"
+			(at 149.86 54.61 0)
+			(hide yes)
+			(show_name no)
+			(do_not_autoplace no)
+			(effects
+				(font
+					(size 1.27 1.27)
+				)
+			)
+		)
 		(pin "1"
 		)
@@
 		(property "Description" ""
 			(at 162.56 40.64 0)
+			(hide yes)
+			(show_name no)
+			(do_not_autoplace no)
+			(effects
+				(font
+					(size 1.27 1.27)
+				)
+			)
+		)
+		(property "LCSC" "C17414"
+			(at 161.0614 44.45 0)
 			(hide yes)
 			(show_name no)
@@
 			(hide yes)
 			(show_name no)
+			(do_not_autoplace no)
+			(effects
+				(font
+					(size 1.27 1.27)
+				)
+			)
+		)
+		(property "LCSC" "C5661"
+			(at 229.235 106.045 0)
+			(hide yes)
+			(show_name no)
