File: Board/fpga_support.kicad_sch (KiCad schematic)
At the start: 5 parts, among them U4 XC6SLX25-CSG324

Commit message: as submitted
Parts:
- U$2: LCSC C5661 -> C5665
Changed lines of the file:
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@@
 			)
 		)
-		(property "LCSC" "C5661"
+		(property "LCSC" "C5665"
 			(at 219.075 99.06 0)
 			(hide yes)
@@
 			)
 		)
-		(property "LCSC" "C5661"
+		(property "LCSC" "C5665"
 			(at 192.405 95.885 0)
 			(hide yes)
@@
 			)
 		)
-		(property "LCSC" "C5661"
+		(property "LCSC" "C5665"
 			(at 229.235 106.045 0)
 			(hide yes)
